File: NewBrain Original KiCad/One.sch (KiCad schematic (older format))
At the start: 96 parts, among them J1 Conn_02x03_Top_Bottom, J2 Conn_02x03_Top_Bottom, J3 Conn_02x03_Top_Bottom, J4 Conn_02x03_Top_Bottom, Q1 Q_PNP_EBC, U1 74LS21, U100 ZTX107, U107 IN914, U109 IN914, U2 74LS21, U410 MC1489N, U411 MC1488N, U414 LM358, U415 HE721A0530, U416 HE751A0510, U417 74LS04, U420 74LS374, U426 74LS86, U431 74LS32, U433 74LS32, U434 74LS86, U435 74LS04, U436 74LS166, U437 74LS08, U438 74LS08, U439 74LS04, U440 74LS02, U441 74LS32, U446 74LS21, U447 74LS393, U448 74LS10, U449 74LS157, U450 74LS04, U451 SN74LS279AN, U453 2716-Memory_EPROM, U454 74LS166, U455 74LS27, U456 74LS32, U457 74LS10, U458 74LS90, U459 74LS32, U460 74LS112, U461 74LS32, U462 74LS32, U463 74LS32, U464 74LS27, U465 74LS11, U466 74LS21, U467 74LS04, U468 74LS393, U469 74LS10, U470 74LS00, U471 74LS11

Commit message: Start sheet TWO.
Signed-off-by: John Bradley <flypie@rocketmail.com>
Parts:
- removed U1: 74LS21, symbol 74xx:74LS112
- removed U2: 74LS21, symbol 74xx:74LS32
- removed unit 5 of U426
- removed unit 5 of U437
- removed unit 5 of U438
- removed unit 5 of U440
- removed unit 5 of U451
- removed unit 2 of U453
- removed unit 4 of U455
- removed unit 5 of U456
- removed unit 4 of U457
Connections:
- wire segments 654 -> 632

Commit message: Next stage of page 2.
Signed-off-by: John Bradley <flypie@rocketmail.com>
Parts:
- added unit 1 of U446
Connections:
- net labels added: 32\40
- wire segments 632 -> 637
Other:
- note added: "Sheet 2"
- moved on the sheet: C1, C10, C124, C132, C133, C2, C3, C4, C5, C6, C7, C72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

Commit message: Complete most of drawing 2.
Signed-off-by: John Bradley <flypie@rocketmail.com>
Parts:
- added unit 2 of U449
- added unit 5 of U449
- C103: renamed from C4; value C -> 680pf; footprint (none) -> Capacitor_THT:C_Disc_D3.0mm_W1.6mm_P2.50mm
- C104: renamed from C1; value CP -> 47uf; footprint (none) -> Capacitor_THT:C_Disc_D3.0mm_W1.6mm_P2.50mm
- C118: renamed from C8; value C -> 0.1uf; footprint (none) -> Capacitor_THT:C_Disc_D3.0mm_W1.6mm_P2.50mm
- C119: renamed from C7; value CP -> 47uf; footprint (none) -> Capacitor_THT:C_Disc_D3.0mm_W1.6mm_P2.50mm
- C120: renamed from C6; value C -> 0.1; footprint (none) -> Capacitor_THT:C_Disc_D3.0mm_W1.6mm_P2.50mm
- C124, C132, C133, C72, C73: footprint (none) -> Capacitor_THT:C_Disc_D3.0mm_W1.6mm_P2.50mm
- C82: renamed from C10; value C -> 0.47uf; footprint (none) -> Capacitor_THT:C_Disc_D3.0mm_W1.6mm_P2.50mm
- C85: renamed from C9; value C -> 0.47uf; footprint (none) -> Capacitor_THT:C_Disc_D3.0mm_W1.6mm_P2.50mm
- C87: renamed from C3; value C -> 10nf; footprint (none) -> Capacitor_THT:C_Disc_D3.0mm_W1.6mm_P2.50mm
- C89: renamed from C2; value C -> 10nf; footprint (none) -> Capacitor_THT:C_Disc_D3.0mm_W1.6mm_P2.50mm
- C90: renamed from C5; value C -> 0.33uf; footprint (none) -> Capacitor_THT:C_Disc_D3.0mm_W1.6mm_P2.50mm
- J1, J2, J3, J4: footprint (none) -> Connector_PinHeader_2.54mm:PinHeader_2x03_P2.54mm_Vertical
- L117: footprint (none) -> Inductor_THT:L_Axial_L5.0mm_D3.6mm_P10.00mm_Horizontal_Murata_BL01RN1A2A2
- Q1, U107, U109: footprint (none) -> Package_TO_SOT_THT:TO-92_Inline
- Q100: renamed from U100; footprint (none) -> Package_TO_SOT_THT:TO-92_Inline
- R101: renamed from R6; value R -> 10M; footprint (none) -> Resistor_THT:R_Axial_DIN0204_L3.6mm_D1.6mm_P1.90mm_Vertical
- R102: renamed from R1; value R -> 1K; footprint (none) -> Resistor_THT:R_Axial_DIN0204_L3.6mm_D1.6mm_P1.90mm_Vertical
- R105: renamed from R17; value R -> 43; footprint (none) -> Resistor_THT:R_Axial_DIN0204_L3.6mm_D1.6mm_P1.90mm_Vertical
- R106: renamed from R5; value R -> 1K; footprint (none) -> Resistor_THT:R_Axial_DIN0204_L3.6mm_D1.6mm_P1.90mm_Vertical
- R108: renamed from R7; value R -> 15k; footprint (none) -> Resistor_THT:R_Axial_DIN0204_L3.6mm_D1.6mm_P1.90mm_Vertical
- R114: renamed from R2; value R -> 15k; footprint (none) -> Resistor_THT:R_Axial_DIN0204_L3.6mm_D1.6mm_P1.90mm_Vertical
- R116: renamed from R16; value R -> 68; footprint (none) -> Resistor_THT:R_Axial_DIN0204_L3.6mm_D1.6mm_P1.90mm_Vertical
- R121: renamed from R15; value R -> 270; footprint (none) -> Resistor_THT:R_Axial_DIN0204_L3.6mm_D1.6mm_P1.90mm_Vertical
- R122: renamed from R14; value R -> 75; footprint (none) -> Resistor_THT:R_Axial_DIN0204_L3.6mm_D1.6mm_P1.90mm_Vertical
- R123, R13, R131, R22: footprint (none) -> Resistor_THT:R_Axial_DIN0204_L3.6mm_D1.6mm_P1.90mm_Vertical
- R61: value 22K -> 22k; footprint (none) -> Resistor_THT:R_Axial_DIN0204_L3.6mm_D1.6mm_P1.90mm_Vertical
- R74, R75: footprint (none) -> Potentiometer_THT:3362H1103LF
- R76: renamed from R11; value R -> 22k; footprint (none) -> Resistor_THT:R_Axial_DIN0204_L3.6mm_D1.6mm_P1.90mm_Vertical
- R77: renamed from R12; value R -> 10; footprint (none) -> Resistor_THT:R_Axial_DIN0204_L3.6mm_D1.6mm_P1.90mm_Vertical
- R78: renamed from R9; value R -> 22k; footprint (none) -> Resistor_THT:R_Axial_DIN0204_L3.6mm_D1.6mm_P1.90mm_Vertical
- R79: renamed from R10; value R -> 10; footprint (none) -> Resistor_THT:R_Axial_DIN0204_L3.6mm_D1.6mm_P1.90mm_Vertical
- R83: renamed from R20; value R -> 47; footprint (none) -> Resistor_THT:R_Axial_DIN0204_L3.6mm_D1.6mm_P1.90mm_Vertical
- R84: renamed from R21; value R -> 3.3; footprint (none) -> Resistor_THT:R_Axial_DIN0204_L3.6mm_D1.6mm_P1.90mm_Vertical
- R86: renamed from R19; value R -> 47; footprint (none) -> Resistor_THT:R_Axial_DIN0204_L3.6mm_D1.6mm_P1.90mm_Vertical
- R92: renamed from R8; value R -> 47K; footprint (none) -> Resistor_THT:R_Axial_DIN0204_L3.6mm_D1.6mm_P1.90mm_Vertical
- R97: renamed from R18; value R -> 33; footprint (none) -> Resistor_THT:R_Axial_DIN0204_L3.6mm_D1.6mm_P1.90mm_Vertical
- R98: renamed from R4; value R -> 39k; footprint (none) -> Resistor_THT:R_Axial_DIN0204_L3.6mm_D1.6mm_P1.90mm_Vertical
- R99: renamed from R3; value R -> 39k; footprint (none) -> Resistor_THT:R_Axial_DIN0204_L3.6mm_D1.6mm_P1.90mm_Vertical
- U414: footprint (none) -> Package_DIP:DIP-8_W7.62mm
- U417: value 74LS04 -> MC14584BDG; footprint (none) -> Package_DIP:DIP-14_W7.62mm; symbol 74xx:74LS04 -> SamacSys_Parts:MC14584BDG_UNITS
- U420: footprint (none) -> Package_DIP:DIP-20_W7.62mm
- U426, U431, U433, U434, U437, U438, U439, U440, U446, U447, U448, U450, U455, U456, U457, U458, U459, U462, U463, U465, U466, U467, U468, U469, U470, U471: footprint (none) -> Package_DIP:DIP-14_W7.62mm
- U435: value 74LS04 -> 74LS06; footprint (none) -> Package_DIP:DIP-14_W7.62mm
- U435: value 74LS04 -> 74LS06; footprint (none) -> Package_DIP:DIP-14_W7.62mm; symbol 74xx:74LS04 -> 74xx:74LS06
- U436, U454, U460: footprint (none) -> Package_DIP:DIP-16_W7.62mm
- U440: renamed from U439; value 74LS04 -> 74LS02; footprint (none) -> Package_DIP:DIP-14_W7.62mm; symbol 74xx:74LS04 -> 74xx:74LS02
- U441: value 74LS32 -> 74LS00; footprint (none) -> Package_DIP:DIP-14_W7.62mm; symbol 74xx:74LS04 -> 74xx:74LS00
- U449: footprint (none) -> Package_DIP:DIP-16_W7.62mm; symbol 74xx:74LS157 -> 74xx:74LS157_UNITS
- U450: renamed from U439; footprint (none) -> Package_DIP:DIP-14_W7.62mm
- U451: footprint DIP794W53P254L1930H508Q16N -> Package_DIP:DIP-16_W7.62mm
- U461: value 74LS32 -> 74LS95; footprint (none) -> Package_DIP:DIP-14_W7.62mm
- U464: value 74LS27 -> 74LS11; footprint (none) -> Package_DIP:DIP-14_W7.62mm
Connections:
- net labels added: DB-0, DB-1, DB-2, DB-3, DB-4, DB-5, DB-6, DB-7, V0
- net labels removed: DA-0, DA-1, DA-2, DA-3, DA-4, DA-5, DA-6, DA-7
- wire segments 637 -> 645
- no-connect marks 3 -> 13

Commit message: Minor label changes.
Signed-off-by: John Bradley <flypie@rocketmail.com>
Connections:
- net AB-8: no longer U453.23 (A8), U456.3
- net at U447.11 (Q0): now also U446.4, U448.10, U448.2, U464.2
- net AB-10: no longer names the net of U453.19 (A10), U456.8
- net AB-9: no longer names the net of U453.22 (A9), U456.11
- new net: U453.23 (A8), U456.3
- no-connect marks 13 -> 17
Changed lines of the file:
@@
 	1825 2725 1825 2575
 $Comp
-L 2732-memory_eprom:2716-Memory_EPROM U453
-U 1 1 5EFE9032
-P 1575 4925
-F 0 "U453" H 1875 5050 59  0000 C CNN
-F 1 "2716-Memory_EPROM" H 1625 5425 59  0001 L BNN
-F 2 "Package_DIP:DIP-24_W10.16mm_LongPads" H 1625 6025 50  0001 C CNN
-F 3 "" H 1975 4175 50  0001 C CNN
-	1    1575 4925
-	1    0    0    -1
-$EndComp
-$Comp
 L 74xx:74LS32 U456
 U 1 1 5F00A0E2
@@
 Wire Wire Line
 	1375 5025 1150 5025
-Text Label 1150 5025 0    50   ~ 0
-AB-0
 Wire Wire Line
 	1375 5125 1150 5125
@@
 AB-6
 Wire Wire Line
-	1375 5725 1150 5725
-Text Label 1150 5725 0    50   ~ 0
-AB-7
-Wire Wire Line
-	1375 5825 1150 5825
-Text Label 1150 5825 0    50   ~ 0
-AB-8
-Wire Wire Line
-	1375 5925 1150 5925
-Text Label 1150 5925 0    50   ~ 0
-AB-9
-Wire Wire Line
-	1375 6025 1150 6025
-Text Label 1150 6025 0    50   ~ 0
-AB-10
-Wire Wire Line
-	3450 4075 3450 4300
-Text Label 3450 4300 1    50   ~ 0
-AB-8
-Wire Wire Line
-	2900 4050 2900 4275
-Text Label 2900 4275 1    50   ~ 0
-AB-9
-Wire Wire Line
 	2250 4075 2250 4300
-Text Label 2250 4300 1    50   ~ 0
-AB-10
 Text Label 2600 5025 2    50   ~ 0
 DB-0
@@
 Wire Wire Line
 	6200 2525 5975 2525
-Text Label 5975 2525 0    50   ~ 0
-AB-8
 Wire Wire Line
 	6800 2625 6800 4875
@@
 Wire Wire Line
 	13100 2175 13100 1975
-Text Label 13100 1975 1    50   ~ 0
-RD7
 Wire Wire Line
 	13000 2175 13000 1975
-Text Label 13000 1975 1    50   ~ 0
-RD6
 Wire Wire Line
 	12900 2175 12900 1975
-Text Label 12900 1975 1    50   ~ 0
-RD3
 Wire Wire Line
 	12800 2175 12800 1975
-Text Label 12800 1975 1    50   ~ 0
-RD2
 Wire Wire Line
 	12700 2175 12700 1975
-Text Label 12700 1975 1    50   ~ 0
-RD0
 Wire Wire Line
 	12600 2175 12600 1975
-Text Label 12600 1975 1    50   ~ 0
-RD1
 Wire Wire Line
 	12500 2175 12500 1975
-Text Label 12500 1975 1    50   ~ 0
-RD4
 Wire Wire Line
 	12400 2175 12400 1975
-Text Label 12400 1975 1    50   ~ 0
-RD5
 Wire Wire Line
 	13400 2675 13525 2675
@@
 Wire Wire Line
 	16850 2950 16850 3075
-Text Label 15575 3450 2    50   ~ 0
-TDO
 $Comp
 L power:VCC #PWR0115
@@
 Text Label 18925 1950 2    50   ~ 0
 TPIN
-Text Label 20300 2650 0    50   ~ 0
-TDI
 $Comp
 L Device:D U107
@@
 	6125 6650 6125 7500
 Wire Wire Line
-	8450 5950 8550 5950
-Wire Wire Line
 	8550 5950 8550 6775
 Wire Wire Line
@@
 	19175 7350 19175 7950
 NoConn ~ 18950 8325
-Text Label 17250 8425 2    50   ~ 0
-~TM2
-Text Label 17750 7350 2    50   ~ 0
-~TM1
 $Comp
 L power:VCC #PWR0133
@@
 Wire Wire Line
 	8600 14625 8650 14625
-Text Label 8650 14625 0    50   ~ 0
-~BUSRQ
 Text Label 8650 15025 0    50   ~ 0
 BUSRQ
@@
 NoConn ~ 2700 9325
 NoConn ~ 2700 9225
+Text GLabel 12400 1975 1    50   Input ~ 0
+RD5
+Text GLabel 12500 1975 1    50   Input ~ 0
+RD4
+Text GLabel 12600 1975 1    50   Input ~ 0
+RD1
+Text GLabel 12700 1975 1    50   Input ~ 0
+RD0
+Text GLabel 12800 1975 1    50   Input ~ 0
+RD2
+Text GLabel 12900 1975 1    50   Input ~ 0
+RD3
+Text GLabel 13000 1975 1    50   Input ~ 0
+RD6
+Text GLabel 13100 1975 1    50   Input ~ 0
+RD7
+Text GLabel 8650 14625 2    50   Input ~ 0
+~BUSRQ
+Text GLabel 5975 2525 0    50   Input ~ 0
+AB-8
+Wire Wire Line
+	8425 5950 8550 5950
+NoConn ~ 8425 6050
+NoConn ~ 8425 6150
+NoConn ~ 17250 8225
+NoConn ~ 17250 8525
+Text GLabel 17750 7350 0    50   Input ~ 0
+~TM1
+Text GLabel 17250 8425 0    50   Input ~ 0
+~TM2
+Text GLabel 20300 2650 2    50   Input ~ 0
+TDI
+Text GLabel 15550 3450 0    50   Input ~ 0
+TDO
+Text GLabel 1150 5025 0    50   Input ~ 0
+AB-0
+Text GLabel 1150 5725 0    50   Input ~ 0
+AB-7
+Wire Wire Line
+	1375 5725 1150 5725
+$Comp
+L 2732-memory_eprom:2716-Memory_EPROM U453
+U 1 1 5EFE9032
+P 1575 4925
+F 0 "U453" H 1875 5050 59  0000 C CNN
+F 1 "2716-Memory_EPROM" H 1625 5425 59  0001 L BNN
+F 2 "Package_DIP:DIP-24_W10.16mm_LongPads" H 1625 6025 50  0001 C CNN
+F 3 "" H 1975 4175 50  0001 C CNN
+	1    1575 4925
+	1    0    0    -1
+$EndComp
+Wire Wire Line
+	2250 4300 750  4300
+Wire Wire Line
+	750  4300 750  6025
+Wire Wire Line
+	750  6025 1375 6025
+Wire Wire Line
+	2900 4525 800  4525
+Wire Wire Line
+	800  4525 800  5925
+Wire Wire Line
+	800  5925 1375 5925
+Wire Wire Line
+	2900 4050 2900 4525
+Wire Wire Line
+	3450 4600 850  4600
+Wire Wire Line
+	850  4600 850  5825
+Wire Wire Line
+	850  5825 1375 5825
+Wire Wire Line
+	3450 4075 3450 4600
 $EndSCHEMATC

Commit message: Some more link fixes now below 100 warnings.
Signed-off-by: John Bradley <flypie@rocketmail.com>
Parts:
- removed unit 1 of U446
- removed unit 5 of U449
- U435: renamed from U450; value 74LS04 -> 74LS06
- renumbered J1 to J11, J2 to J12, J3 to J13, J4 to J14
Connections:
- net AB-7 is gone; now on net LAB-7: U453.1 (A7)
- net FPO is gone; now on net FP: U451.11 (3~S1), U471.12
- net 1\8: now also U457.3
- net GR: now also U440.4, U463.1
- net RC3: now also U435.13; no longer U435.11
- net UCR: now also U453.18 (~CE~/PGM)
- net ~GR: now also U440.5, U440.6, U461.2 (P0), U463.11
- net LAB-7: now reaches U420.2 (O0), U437.10, U437.4, U454.2 (A), U455.3
- net at U426.9: now also U435.12; no longer U435.10
- net AB-0 renamed LAB-0
- net AB-1 renamed LAB-1
- net AB-2 renamed LAB-2
- net AB-3 renamed LAB-3
- net AB-4 renamed LAB-4
- net AB-5 renamed LAB-5
- net AB-6 renamed LAB-6
- net AB-8 renamed LAB-8
- net DB-0 renamed LDB-0
- net DB-1 renamed LDB-1
- net DB-2 renamed LDB-2
- net DB-3 renamed LDB-3
- net DB-4 renamed LDB-4
- net DB-5 renamed LDB-5
- net DB-6 renamed LDB-6
- net DB-7 renamed LDB-7
- no-connect marks 17 -> 19
Other:
- note removed: "Sheet 2"

Commit message: More Label fixing. Down to 16 Warnings. Lots of devie Labels and balues wrong.
Signed-off-by: John Bradley <flypie@rocketmail.com>
Parts:
- removed R61: 22k, Resistor_THT:R_Axial_DIN0204_L3.6mm_D1.6mm_P1.90mm_Vertical, symbol Device:R
- added RN66: R_Network03, Resistor_THT:R_Array_SIP5, symbol Device:R_Network03
Connections:
- net LAB-8 is gone; now on net LAB-7: U437.6
- net GND: now also U414.4 (V-); no longer U414.8 (V+)
- net LAB-7: no longer U420.2 (O0), U437.10, U437.4, U454.2 (A), U455.3
- net RC0: now also U447.1 (CP), U458.1 (CP1..3), U470.4
- net V0: now also U414.8 (V+); no longer U414.4 (V-)
- net VCC: now also RN66.1 (common); no longer U411.14 (VCC_+)
- net -12I: now reaches U411.1 (VCC-)
- net at U446.5, U447.13 (CP), U447.6 (Q3)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: no longer U447.5 (Q2), U448.13, U466.13
- net at U450.5, U466.8: now also U463.4
- net BOL renamed 80L
- new net: J12.1 (Pin_1), U410.1 (1A)
- new net: RN66.3 (R2), U410.12 (4CONT)
- new net: RN66.2 (R1), U410.2 (1CONT)
- new net: RN66.4 (R3), U410.9 (3CONT)
- new net: U420.2 (O0), U437.10, U437.4, U454.2 (A), U455.3
- new net: U447.5 (Q2), U448.13, U466.13
- new net +12: U411.14 (VCC_+)
- no-connect marks 19 -> 21
Changed lines of the file:
@@
 Wire Wire Line
 	2000 1450 1050 1450
-Text Label 1050 1450 0    50   ~ 0
-BOL
 Wire Wire Line
 	2000 1650 1075 1650
@@
 	3900 8425 4700 8425
 Wire Wire Line
-	3900 8325 4175 8325
-Wire Wire Line
 	1775 8050 2275 8050
 Wire Wire Line
@@
 L power:VCC #PWR0106
 U 1 1 5EEBA9A4
-P 5200 7525
-F 0 "#PWR0106" H 5200 7375 50  0001 C CNN
-F 1 "VCC" V 5175 7675 50  0000 L CNN
-F 2 "" H 5200 7525 50  0001 C CNN
-F 3 "" H 5200 7525 50  0001 C CNN
-	1    5200 7525
+P 5500 7525
+F 0 "#PWR0106" H 5500 7375 50  0001 C CNN
+F 1 "VCC" V 5475 7675 50  0000 L CNN
+F 2 "" H 5500 7525 50  0001 C CNN
+F 3 "" H 5500 7525 50  0001 C CNN
+	1    5500 7525
 	0    1    1    0
 $EndComp
@@
 Wire Wire Line
 	2600 9425 2700 9425
-Text Label 2600 9475 2    50   ~ 0
-DO
 Wire Wire Line
 	1275 9250 1275 9450
@@
 Wire Wire Line
 	2600 7425 4175 7425
-$Comp
-L Device:R R61
-U 1 1 5EEE0DAF
-P 4600 7525
-F 0 "R61" V 4350 7525 50  0000 C CNN
-F 1 "22k" V 4450 7525 50  0000 C CNN
-F 2 "Resistor_THT:R_Axial_DIN0204_L3.6mm_D1.6mm_P1.90mm_Vertical" V 4530 7525 50  0001 C CNN
-F 3 "~" H 4600 7525 50  0001 C CNN
-	1    4600 7525
-	0    1    1    0
-$EndComp
-Wire Wire Line
-	4750 7525 5200 7525
-Wire Wire Line
-	4175 8325 4175 8025
-Connection ~ 4175 8025
-Wire Wire Line
-	2700 7925 2700 7825
-Connection ~ 2700 7825
-Wire Wire Line
-	2700 7825 2700 7525
-Wire Wire Line
-	2700 7525 4175 7525
-Wire Wire Line
-	4175 7525 4175 8025
-Connection ~ 4175 7525
-Wire Wire Line
-	4175 7525 4450 7525
 Wire Wire Line
 	1775 9250 2000 9250
@@
 	6025 6450 7300 6450
 Wire Wire Line
-	7225 6250 7225 5950
-Wire Wire Line
 	7225 5950 7425 5950
-Wire Wire Line
-	7025 6250 7225 6250
 $Comp
 L 74xx:74LS90 U458
@@
 Wire Wire Line
 	6800 2425 7050 2425
-Text Label 8075 2425 0    50   ~ 0
-FS
 $Comp
 L 74xx:74LS04 U439
@@
 Wire Wire Line
 	19700 2650 20300 2650
-Text Label 18925 1950 2    50   ~ 0
-TPIN
 $Comp
 L Device:D U107
@@
 	7100 7550 7100 8225
 Wire Wire Line
-	7225 8550 7200 8550
-Connection ~ 7225 6250
-Wire Wire Line
 	7575 7750 7575 7675
 Wire Wire Line
-	7575 7675 7225 7675
-Wire Wire Line
-	7225 6250 7225 7675
-Connection ~ 7225 7675
-Wire Wire Line
-	7225 7675 7225 8550
-Wire Wire Line
-	7200 8850 7200 8550
-Wire Wire Line
 	7025 5950 7150 5950
 Wire Wire Line
@@
 Connection ~ 7300 6250
 Wire Wire Line
-	7025 6150 7025 6250
-Wire Wire Line
 	7025 7425 7850 7425
 Wire Wire Line
@@
 Wire Wire Line
 	8250 9275 8250 9775
-Connection ~ 7025 6250
-Wire Wire Line
-	7025 6250 7025 7425
 Wire Wire Line
 	7475 8350 7475 9400
@@
 Wire Wire Line
 	14400 12350 13950 12350
-Text Label 13925 11825 2    50   ~ 0
-~FRMR
 $Comp
 L Device:R R123
@@
 Wire Wire Line
 	14400 12575 14100 12575
-Text Label 14100 12575 2    50   ~ 0
-~CLCLK
 $Comp
 L 74xx:74LS11 U465
@@
 Wire Wire Line
 	15525 12400 15675 12400
-Text Label 15675 12400 0    50   ~ 0
-~CLKINT
 Wire Wire Line
 	15575 9000 15750 9000
@@
 Wire Wire Line
 	15300 7075 16350 7075
-Text Label 16350 8425 0    50   ~ 0
-TVP
 $Comp
 L 74xx:74LS04 U450
@@
 	0    -1   -1   0
 $EndComp
-Wire Wire Line
-	8100 10400 1300 10400
 $Comp
 L 74xx:74LS32 U463
@@
 	1400 11700 1300 11700
 Wire Wire Line
-	1300 10400 1300 11700
-Wire Wire Line
 	2250 11750 2250 11800
 Wire Wire Line
@@
 	2175 10900 4300 10900
 Wire Wire Line
-	5925 10650 2025 10650
+	5925 10650 3925 10650
 Wire Wire Line
 	2025 10650 2025 11550
@@
 L power:GND #PWR0236
 U 1 1 666D723E
-P 17375 2850
-F 0 "#PWR0236" H 17375 2600 50  0001 C CNN
-F 1 "GND" V 17375 2700 50  0000 R CNN
-F 2 "" H 17375 2850 50  0001 C CNN
-F 3 "" H 17375 2850 50  0001 C CNN
-	1    17375 2850
-	1    0    0    -1
+P 17375 2250
+F 0 "#PWR0236" H 17375 2000 50  0001 C CNN
+F 1 "GND" V 17375 2100 50  0000 R CNN
+F 2 "" H 17375 2250 50  0001 C CNN
+F 3 "" H 17375 2250 50  0001 C CNN
+	1    17375 2250
+	-1   0    0    1
 $EndComp
-Text Label 17375 2250 0    50   ~ 0
+Text Label 17375 2850 0    50   ~ 0
 V0
 $Comp
@@
 NoConn ~ 1775 8150
 $Comp
-L power:VCC #PWR0245
-U 1 1 66EF120A
-P 4000 9125
-F 0 "#PWR0245" H 4000 8975 50  0001 C CNN
-F 1 "VCC" H 4025 9325 50  0000 C CNN
-F 2 "" H 4000 9125 50  0001 C CNN
-F 3 "" H 4000 9125 50  0001 C CNN
-	1    4000 9125
-	0    1    1    0
-$EndComp
-$Comp
 L power:VCC #PWR0246
 U 1 1 66EF3F6F
@@
 Text GLabel 4700 9275 2    50   Input ~ 0
 ~RTSD
-Text GLabel 4175 7425 2    50   Input ~ 0
-RDDK
 Text GLabel 4700 9625 2    50   Input ~ 0
 PO
@@
 LAB-0
 Text Label 5975 2525 2    50   ~ 0
-LAB-8
+LAB-7
 $Comp
 L Connector_Generic:Conn_02x03_Top_Bottom J12
@@
 Text GLabel 9925 2575 0    50   Input ~ 0
 RV
-Text Label 11900 4875 0    50   ~ 0
-LAB-7
 Text GLabel 4125 1650 0    50   Input ~ 0
 ~VDLD
@@
 Text GLabel 13550 6175 0    50   Input ~ 0
 GR
+Text GLabel 13925 11825 0    50   Input ~ 0
+~FRMR
+Text GLabel 16350 8425 2    50   Input ~ 0
+TVP
+Text GLabel 15675 12400 2    50   Input ~ 0
+~CLKINT
+Text GLabel 18925 1950 0    50   Input ~ 0
+TPIN
+Text GLabel 2600 9475 0    50   Input ~ 0
+DO
+Text GLabel 14100 12575 0    50   Input ~ 0
+~CLCLK
+NoConn ~ 18425 5900
+NoConn ~ 18450 6725
+Wire Wire Line
+	8100 10375 1300 10375
+Connection ~ 8100 10375
+Wire Wire Line
+	1300 10375 1300 11700
+Text GLabel 1050 1450 0    50   Input ~ 0
+80L
+Text GLabel 8075 2425 2    50   Input ~ 0
+FS
+Wire Wire Line
+	7025 6150 7100 6150
+Wire Wire Line
+	7100 6150 7100 6400
+Wire Wire Line
+	7100 6400 7025 6400
+Wire Wire Line
+	7025 6400 7025 7425
+Wire Wire Line
+	7025 6250 7025 6325
+Wire Wire Line
+	7025 6325 6900 6325
+Wire Wire Line
+	6900 7675 7575 7675
+Wire Wire Line
+	6900 6325 6900 7675
+Wire Wire Line
+	7200 8850 7200 8475
+Wire Wire Line
+	7200 8475 6900 8475
+Wire Wire Line
+	6900 8475 6900 7675
+Connection ~ 6900 7675
+Wire Wire Line
+	7025 6250 7225 6250
+Wire Wire Line
+	7225 6250 7225 5950
+Connection ~ 7025 6250
+Wire Wire Line
+	3925 11450 3925 10650
+Connection ~ 3925 11450
+Connection ~ 3925 10650
+Wire Wire Line
+	3925 10650 2025 10650
+Text Label 4175 7425 0    50   ~ 0
+RDDK
+Wire Wire Line
+	2700 7925 2500 7925
+Wire Wire Line
+	2500 7925 2500 7525
+$Comp
+L Device:R_Network03 RN66
+U 1 1 62260EA2
+P 5300 7625
+F 0 "RN66" V 4925 7625 50  0000 C CNN
+F 1 "R_Network03" V 5025 7625 50  0000 C CNN
+F 2 "Resistor_THT:R_Array_SIP5" V 5575 7625 50  0001 C CNN
+F 3 "http://www.vishay.com/docs/31509/csc.pdf" H 5300 7625 50  0001 C CNN
+	1    5300 7625
+	0    1    1    0
+$EndComp
+Wire Wire Line
+	5100 7625 4175 7625
+Wire Wire Line
+	4175 7625 4175 8025
+Wire Wire Line
+	2500 7525 5100 7525
+Wire Wire Line
+	4375 8325 4375 7725
+Wire Wire Line
+	4375 7725 5100 7725
+Wire Wire Line
+	3900 8325 4375 8325
+Text GLabel 4000 9125 2    50   Input ~ 0
++12
+Text GLabel 2700 9125 0    50   Input ~ 0
+-12I
 $EndSCHEMATC
