File: NewBrain Original KiCad/One.sch (KiCad schematic (older format))
At the start: 94 parts, among them J11 Conn_02x03_Top_Bottom, J12 Conn_02x03_Top_Bottom, J13 Conn_02x03_Top_Bottom, J14 Conn_02x03_Top_Bottom, Q1 Q_PNP_EBC, Q100 ZTX107, U107 IN914, U109 IN914, U410 MC1489N, U411 MC1488N, U414 LM358, U415 HE721A0530, U416 HE751A0510, U417 MC14584BDG, U420 74LS374, U426 74LS86, U431 74LS32, U433 74LS32, U434 74LS86, U435 74LS06, U436 74LS166, U437 74LS08, U438 74LS08, U439 74LS04, U440 74LS02, U441 74LS00, U446 74LS21, U447 74LS393, U448 74LS10, U449 74LS157, U450 74LS04, U451 SN74LS279AN, U453 2716-Memory_EPROM, U454 74LS166, U455 74LS27, U456 74LS32, U457 74LS10, U458 74LS90, U459 74LS32, U460 74LS112, U461 74LS95, U462 74LS32, U463 74LS32, U464 74LS11, U465 74LS11, U466 74LS21, U467 74LS04, U468 74LS393, U469 74LS10, U470 74LS00, U471 74LS11

Commit message: Resolve inconsistencies in circuit diagram buy following traces.
Resistor name used twice temp solution add a and b to name.

Signed-off-by: John Bradley <flypie@rocketmail.com>
Parts:
- Q110: renamed from Q1; value Q_PNP_EBC -> ZTC212
- R81: renamed from R22; value R -> 3.3
- renumbered R13 to R71
Connections:
- net CRDO is gone; now on net LDB-0: U426.10
- net V0 renamed V0A
Other:
- note added: "CRD0 on schematic. LDB-0 following traces."
Changed lines of the file:
@@
 Wire Wire Line
 	2700 2100 2525 2100
-Text Label 1075 2100 0    50   ~ 0
-RC3
 Wire Wire Line
 	2700 2300 2375 2300
 Text Label 2375 2300 0    50   ~ 0
-CRDO
+LDB-0
 Wire Wire Line
 	3625 2000 3375 2000
@@
 Wire Wire Line
 	3550 3475 3550 3050
-Text Label 2350 3050 0    50   ~ 0
-RC2
-Text Label 3000 3050 0    50   ~ 0
-RC1
-Text Label 3550 3050 0    50   ~ 0
-RC0
 Wire Wire Line
 	1375 5025 1150 5025
@@
 Text Label 1100 7000 0    50   ~ 0
 TXT
-Text Label 1100 7200 0    50   ~ 0
-UCR
 Wire Wire Line
 	4125 6225 3900 6225
@@
 	2400 7825 2700 7825
 Wire Wire Line
-	2700 8025 2600 8025
-Wire Wire Line
-	2600 8025 2600 7425
-Wire Wire Line
-	2600 7425 4175 7425
-Wire Wire Line
 	1775 9250 2000 9250
 Wire Wire Line
@@
 Wire Wire Line
 	7575 3625 7325 3625
-Text Label 7325 3625 2    50   ~ 0
-TVSD
 $Comp
 L 74xx:74LS08 U438
@@
 Wire Wire Line
 	8100 6850 8300 6850
-Text Label 8300 6850 2    50   ~ 0
-UCR
 Connection ~ 7300 6250
 Wire Wire Line
@@
 $EndComp
 $Comp
-L Device:Q_PNP_EBC Q1
+L Device:Q_PNP_EBC Q110
 U 1 1 619E4661
 P 19000 10575
-F 0 "Q1" H 19225 10525 50  0000 L CNN
-F 1 "Q_PNP_EBC" H 19225 10575 50  0000 L CNN
+F 0 "Q110" H 19225 10525 50  0000 L CNN
+F 1 "ZTC212" H 19225 10575 50  0000 L CNN
 F 2 "Package_TO_SOT_THT:TO-92_Inline" H 19200 10675 50  0001 C CNN
 F 3 "~" H 19000 10575 50  0001 C CNN
@@
 Text Label 19350 10800 0    50   ~ 0
 CMPVID
-Text Label 19350 11425 0    50   ~ 0
-K12
-Text Label 19350 11125 0    50   ~ 0
-K11
 $Comp
 L power:GND #PWR0132
@@
 	19450 8275 19450 8225
 $Comp
-L Device:R R22
+L Device:R R81
 U 1 1 62339463
 P 19600 8225
-F 0 "R22" V 19850 8200 50  0000 C CNN
-F 1 "R" V 19750 8200 50  0000 C CNN
+F 0 "R81" V 19850 8200 50  0000 C CNN
+F 1 "3.3" V 19750 8200 50  0000 C CNN
 F 2 "Resistor_THT:R_Axial_DIN0204_L3.6mm_D1.6mm_P1.90mm_Vertical" V 19530 8225 50  0001 C CNN
 F 3 "~" H 19600 8225 50  0001 C CNN
@@
 Wire Wire Line
 	1200 12775 1200 13050
-Text Label 1200 13050 0    50   ~ 0
-UCR
 Wire Wire Line
 	3250 11750 3250 12875
@@
 	3250 12875 3250 13075
 Connection ~ 3250 12875
-Text Label 3250 13075 0    50   ~ 0
-RC3
 Wire Wire Line
 	3250 11650 3475 11650
@@
 Wire Wire Line
 	3925 11450 3925 13075
-Text Label 3475 13075 0    50   ~ 0
-RC2
-Text Label 3700 13075 0    50   ~ 0
-RC1
-Text Label 3925 13075 0    50   ~ 0
-RC0
 Wire Wire Line
 	2250 11450 2175 11450
@@
 $EndComp
 $Comp
-L Device:R R13
+L Device:R R71
 U 1 1 62A6BC14
 P 4975 11650
-F 0 "R13" H 5075 11700 50  0000 L CNN
+F 0 "R71" H 5075 11700 50  0000 L CNN
 F 1 "470" H 5075 11650 50  0000 L CNN
 F 2 "Resistor_THT:R_Axial_DIN0204_L3.6mm_D1.6mm_P1.90mm_Vertical" V 4905 11650 50  0001 C CNN
@@
 	-1   0    0    1
 $EndComp
-Text Label 17375 2850 0    50   ~ 0
-V0
 $Comp
 L power:GND #PWR0243
@@
 1\8
 Wire Wire Line
-	5575 2275 28000 2275
-Wire Wire Line
-	28000 2275 28000 18525
-Wire Wire Line
 	3325 1350 3200 1350
 Wire Wire Line
@@
 Wire Wire Line
 	3925 10650 2025 10650
-Text Label 4175 7425 0    50   ~ 0
-RDDK
 Wire Wire Line
 	2700 7925 2500 7925
@@
 Text GLabel 2700 9125 0    50   Input ~ 0
 -12I
+Text GLabel 1100 7200 0    50   Input ~ 0
+UCR
+Text GLabel 8300 6850 2    50   Input ~ 0
+UCR
+Text GLabel 1200 13050 2    50   Input ~ 0
+UCR
+Text GLabel 7325 3625 0    50   Input ~ 0
+TVSD
+Text GLabel 19350 11125 2    50   Input ~ 0
+K11
+Text GLabel 19350 11425 2    50   Input ~ 0
+K12
+Text GLabel 3925 13075 2    50   Input ~ 0
+RC0
+Text GLabel 3700 13075 2    50   Input ~ 0
+RC1
+Text GLabel 3475 13075 2    50   Input ~ 0
+RC2
+Text GLabel 3250 13075 2    50   Input ~ 0
+RC3
+Text GLabel 3550 3050 2    50   Input ~ 0
+RC0
+Text GLabel 3000 3050 2    50   Input ~ 0
+RC1
+Text GLabel 2350 3050 2    50   Input ~ 0
+RC2
+Text GLabel 1075 2100 0    50   Input ~ 0
+RC3
+Text Notes 2400 2450 0    50   ~ 0
+CRD0 on schematic.  LDB-0 following traces.
+Text GLabel 2700 8025 0    50   Input ~ 0
+RDDK
+Text GLabel 17375 2850 2    50   Input ~ 0
+V0A
 $EndSCHEMATC
