File: NewBrain Original KiCad/Two.sch (KiCad schematic (older format))
At the start: 0 parts

Commit message: Next stage of page 2.
Signed-off-by: John Bradley <flypie@rocketmail.com>
Parts:
- added C18: 0.1, symbol Device:C
- added C64, C? (x7): 33pf, symbol Device:C
- added C94, C95, C? (x2): 47uf, symbol Device:CP
- added C? (x3): CP, symbol Device:CP
- added D1: 1N4733A, symbol Device:D_Zener
- added D24, D31: IN4001, symbol Device:D
- added D93, D96: 1N4148, symbol Device:D
- added PWRIN1: Conn_02x03_Counter_Clockwise, symbol Connector_Generic:Conn_02x03_Counter_Clockwise
- added Q17: ZTX650, symbol Device:Q_NPN_CBE
- added Q20: ZTX107, symbol Device:Q_NPN_EBC
- added Q66: 2N3906, Package_TO_SOT_THT:TO-92_Inline, symbol Transistor_BJT:2N3906
- added Q8, Q?: 2n5193, Package_TO_SOT_THT:TO-126-3_Vertical, symbol Device:Q_PNP_ECB
- added R112: 1K0, symbol Device:R
- added R113, R? (x2): 4K7, symbol Device:R
- added R2: 820, symbol Device:R
- added R5: 220, symbol Device:R
- added R6, R? (x8): 4k7, symbol Device:R
- added R60: 1K, symbol Device:R
- added R62: 12k, symbol Device:R
- added R63, R? (x10): 22, symbol Device:R
- added R? (x2): 32, symbol Device:R
- added U401: LM358, symbol Amplifier_Operational:LM358
- added U402, U403, U404, U405: 74LS153, symbol 74xx:74LS153
- added U406: 2764, Package_DIP:DIP-28_W15.24mm, symbol Memory_EPROM:2764
- added U407: NEC-PD2364, Package_DIP:DIP-28_W15.24mm, symbol local:NEC-PD2364
- added U408: NEC-PD23128, Package_DIP:DIP-28_W15.24mm, symbol local:NEC-PD23128
- added U409: Z80CPU-DIP, Zilog Z80 Microprocessor 8bit CISC 40-Pin PDIP, symbol Zilog_Z80:Z80CPU-DIP
- added U417, U?: 74LS14, symbol 74xx:74LS14
- added U418: 74LS00, symbol 74xx:74LS00
- added U419: COP420L, Package_DIP:DIP-28_W7.62mm, symbol MCU_COPS:COP420L
- added U422, U423, U424: 74LS161, symbol 74xx:74LS161
- added U425: 74LS74, symbol 74xx:74LS74
- added U429, U432: 74LS04, symbol 74xx:74LS04
- added U431, U462, U?: 74LS32, symbol 74xx:74LS32
- added U443, U465: 74LS11, symbol 74xx:74LS11
- added U444: 74LS157, symbol 74xx:74LS157
- added U445: 74LS112, symbol 74xx:74LS112
- added U452: 74LS04, symbol SamacSys_Parts:MC14584BDG
- added U464: 74LS27, symbol 74xx:74LS27
- added U468: 74LS08, symbol 74xx:74LS08
- added U?: 74LS04, symbol local:ZN404
- added U?: 74LS04, symbol 74xx:74LS245
- added U?: 74LS04, symbol 74xx:74LS32
Connections:
- net labels added: +12, +12I, +5, +5I, -12I, -5v, 1\16, 32A, 33E, 64A, 80L, A15G, AB-0, AB-1, AB-10, AB-11, AB-12, AB-13, AB-14, AB-15, AB-2, AB-3, AB-4, AB-5, AB-6, AB-7, AB-8, AB-9, AB0, CPRQ, DA-0, DA-1, DA-2, DA-3, DA-4, DA-5, DA-6, DA-7, GND, GO, GRND, K1, K10, K2, K3, K4, K5, K6, K7, K8, K9, PWRUP, RAMINH, RC1, RC2, RC3, RCO, ROW, TDI, TDO, TVAD, UCR, VCC, ~COP, ~COPINT, ~FRMR, ~IOREQ, ~MREQ, ~RAMENB, ~RD, ~RFRSH, ~TM1, ~TM2, ~TVCLK, ~TVL, ~WR
- wire segments 0 -> 553

Commit message: Complete most of drawing 2.
Signed-off-by: John Bradley <flypie@rocketmail.com>
Parts:
- removed U444: 74LS157, symbol 74xx:74LS157
- removed U452: 74LS04, symbol SamacSys_Parts:MC14584BDG
- removed unit 4 of U464
- removed unit 4 of U465
- added C17, C19: 33pf, Capacitor_THT:C_Disc_D3.0mm_W1.6mm_P2.50mm, symbol Device:C
- added C44: 0.1uf, Capacitor_THT:C_Disc_D3.0mm_W1.6mm_P2.50mm, symbol Device:C
- added Q49: BC546, Package_TO_SOT_THT:TO-92_Inline, symbol Transistor_BJT:BC546
- added R23: 1K, Resistor_THT:R_Axial_DIN0204_L3.6mm_D1.6mm_P1.90mm_Vertical, symbol Device:R
- added R24, R25, R26, R36, R40, R41, R45, R54: 4K7, Resistor_THT:R_Axial_DIN0204_L3.6mm_D1.6mm_P1.90mm_Vertical, symbol Device:R
- added RN134: R_Network08, Resistor_THT:R_Array_SIP9, symbol Device:R_Network08
- added U412, U428: 74LS257, Package_DIP:DIP-16_W7.62mm, symbol 74xx:74LS257
- added U413, U427: 74LS174, Package_DIP:DIP-16_W7.62mm, symbol 74xx:74LS174
- added unit 1 of U425
- added U426: 74LS86, Package_DIP:DIP-14_W7.62mm, symbol 74xx:74LS86
- added U429: 74LS139, Package_DIP:DIP-16_W7.62mm, symbol 74xx:74LS139
- added U430, U442: 74LS138, Package_DIP:DIP-16_W7.62mm, symbol 74xx:74LS138
- added unit 5 of U432
- added unit 6 of U432
- added unit 1 of U432
- added U433: 74LS32, Package_DIP:DIP-14_W7.62mm, symbol 74xx:74LS32
- added U435: 74LS06, Package_DIP:DIP-14_W7.62mm, symbol 74xx:74LS06
- added unit 2 of U439
- added U441, U470: 74LS00, Package_DIP:DIP-14_W7.62mm, symbol 74xx:74LS00
- added U444: 74LS157_UNITS, Package_DIP:DIP-16_W7.62mm, symbol 74xx:74LS157_UNITS
- added U452: MC14584BDG_UNITS, Package_DIP:DIP-14_W7.62mm, symbol SamacSys_Parts:MC14584BDG_UNITS
- added U460: 74LS112, Package_DIP:DIP-16_W7.62mm, symbol 74xx:74LS112
- added X48: Crystal, Crystal:Crystal_HC52-6mm_Vertical, symbol Device:Crystal
- C11, C12, C14, C15, C16, C20, C21: renamed from C?; footprint (none) -> Capacitor_THT:C_Disc_D3.0mm_W1.6mm_P2.50mm
- C125, C127: renamed from C?; value 47uf -> 10uf; footprint (none) -> Capacitor_THT:C_Disc_D3.0mm_W1.6mm_P2.50mm
- C13, C22, C23: renamed from C?; footprint (none) -> Capacitor_THT:CP_Radial_D4.0mm_P1.50mm
- C18, C64, C94, C95: footprint (none) -> Capacitor_THT:C_Disc_D3.0mm_W1.6mm_P2.50mm
- D1, D24, D31, D93, D96: footprint (none) -> Diode_THT:D_DO-34_SOD68_P2.54mm_Vertical_AnodeUp
- D21: renamed from U?; value 74LS04 -> ZN404; footprint (none) -> Package_TO_SOT_THT:TO-18-2
- PWRIN1: footprint (none) -> Connector_PinHeader_2.54mm:PinHeader_2x03_P2.54mm_Vertical
- Q17, Q20: footprint (none) -> Package_TO_SOT_THT:TO-92_Inline
- R112, R113, R2, R6, R60, R62, R63: footprint (none) -> Resistor_THT:R_Axial_DIN0204_L3.6mm_D1.6mm_P1.90mm_Vertical
- R128: renamed from R?; value 4K7 -> 220K; footprint (none) -> Resistor_THT:R_Axial_DIN0204_L3.6mm_D1.6mm_P1.90mm_Vertical
- R129: renamed from R?; value 4K7 -> 560K; footprint (none) -> Resistor_THT:R_Axial_DIN0204_L3.6mm_D1.6mm_P1.90mm_Vertical
- R27, R28, R29, R30, R31, R32, R33, R34, R35, R37, R38, R39, R42, R43, R44, R46, R47, R48, R49, R50: renamed from R?; footprint (none) -> Resistor_THT:R_Axial_DIN0204_L3.6mm_D1.6mm_P1.90mm_Vertical
- R65: renamed from R5; footprint (none) -> Resistor_THT:R_Axial_DIN0204_L3.6mm_D1.6mm_P1.90mm_Vertical
- U401: footprint (none) -> Package_DIP:DIP-8_W7.62mm
- U402, U403, U404, U405, U422, U423, U424, U445: footprint (none) -> Package_DIP:DIP-16_W7.62mm
- U409: footprint Zilog Z80 Microprocessor 8bit CISC 40-Pin PDIP -> Package_DIP:DIP-40_W15.24mm
- U417: value 74LS14 -> MC14584BDG; footprint (none) -> Package_DIP:DIP-14_W7.62mm; symbol 74xx:74LS14 -> SamacSys_Parts:MC14584BDG_UNITS
- U417: value 74LS14 -> MC14584BDG; footprint (none) -> Package_DIP:DIP-14_W7.62mm
- U418, U425, U431, U432, U443, U462, U465: footprint (none) -> Package_DIP:DIP-14_W7.62mm
- U421: renamed from U?; value 74LS04 -> 74LS06; footprint (none) -> Package_DIP:DIP-20_W7.62mm
- U432: renamed from U?; value 74LS14 -> 74LS04; footprint (none) -> Package_DIP:DIP-14_W7.62mm; symbol 74xx:74LS14 -> 74xx:74LS04
- U438: renamed from U468; footprint (none) -> Package_DIP:DIP-14_W7.62mm
- U439: renamed from U429; footprint (none) -> Package_DIP:DIP-14_W7.62mm
- U459: renamed from U?; value 74LS04 -> 74LS32; footprint (none) -> Package_DIP:DIP-14_W7.62mm
- U462: renamed from U?; footprint (none) -> Package_DIP:DIP-14_W7.62mm
- U464: value 74LS27 -> 74LS11; footprint (none) -> Package_DIP:DIP-14_W7.62mm
- gave numbers to parts that had none: 1
Connections:
- net labels added: 1.3M, 1.4M, 1.5M, 1.6M, 1\8, 1\8c, 3.4M, 3.5M, 3.6M, AB-15G, AB1, AB2, AB3, AB4, AD1, CIA, CTR, D0, DB-0, DB-1, DB-2, DB-3, DB-4, DB-5, DB-6, DB-7, EXP0, EXP1, EXRM0, EXRM1, EXRM2, F5, P0, PR, PRTOV, RD0, RD1, RD2, RD3, RD4, RD5, RD6, RD7, RMSL, RV, TPIN, TVP, ~1\16, ~32\40, ~AB-14M, ~ANIN, ~BUSAK, ~BUSRQ, ~CKVSR, ~CLCLK, ~CLCSA, ~CLDMA, ~CLK, ~CLKINT, ~COG, ~CPRQG, ~CTSD, ~CTSP, ~ENRG, ~ENRG1, ~ENRG2, ~EXP1, ~EXP2, ~HALT, ~INT, ~IORQ, ~M1, ~NMI, ~RESET, ~RFSH, ~ROM0, ~ROM1, ~ROM2, ~ROMOV, ~RST, ~RTSD, ~TVCTL, ~TVTL, ~USER, ~UST, ~VDLD, ~VST, ~WAIT
- net labels removed: A15G, DA-0, DA-1, DA-2, DA-3, DA-4, DA-5, DA-6, DA-7
- wire segments 553 -> 698
- no-connect marks 0 -> 6
Other:
- moved on the sheet: C11, C12, C125, C127, C13, C14, C15, C16, C18, C20, C21, C22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

Commit message: Minor label changes.
Signed-off-by: John Bradley <flypie@rocketmail.com>
Connections:
- net 33E is gone; now on net ~M1: U409.27 (M1)
- net AB1 is gone; now on net AB-1: U429.13 (A1), U429.3 (A1)
- net AB2 is gone; now on net AB-2: U430.1 (A0)
- net AB3 is gone; now on net AB-3: U430.2 (A1)
- net AB4 is gone; now on net AB-4: U430.3 (A2)
- net D0 is gone; now on net DB-0: U413.7 (Q2)
- net EXP1 is gone; now on net ~EXP1: U430.14 (O1)
- net GRND is gone; now on net GND: C22.2, C23.2, D1.1 (K), D21.2 (-), D24.1 (K), D31.1 (K), PWRIN1.5 (Pin_5), R32.2, R33.2, R43.2, R46.2
- net ~COG is gone; now on net ~COP: U429.10 (O2)
- net ~EXP2 is gone; now on net ~EXP0: U429.1 (E)
- net ~IORQ is gone; now on net ~IOREQ: U430.4 (E1)
- net ~RFRSH is gone; now on net ~RFSH: U442.6 (E3), U465.9
- net ~RST is gone; now on net ~RESET: U413.1 (~Mr)
- net AB-0: now also U429.14 (A0), U429.2 (A0)
- net AB0: no longer U429.14 (A0), U429.2 (A0)
- net GND: now also U421.10 (GND), U442.8 (GND)
- net EXP0 renamed ~EXP0
- net P0 renamed PO
- net ~CLCSA renamed ~CLUSA
- no-connect marks 6 -> 15
Changed lines of the file:
@@
 	6750 1475 6425 1475
 Text Label 5825 1375 2    50   ~ 0
-~RFRSH
+~RFSH
 Text Label 5825 1475 2    50   ~ 0
 AB-15G
@@
 	0    1    1    0
 $EndComp
-Text Label 6750 1575 2    50   ~ 0
-~MREQ
 Text Label 6750 1675 2    50   ~ 0
 RAMINH
@@
 Wire Wire Line
 	22275 5775 22350 5775
-Text Label 22350 5500 1    50   ~ 0
-33E
 Wire Wire Line
 	22275 5875 22450 5875
@@
 Wire Wire Line
 	21850 10650 22175 10650
-Text Label 21300 10650 2    50   ~ 0
-GRND
 Wire Wire Line
 	19275 5800 19425 5800
-Text Label 19425 5800 0    50   ~ 0
-GRND
 Wire Wire Line
 	23500 9850 23500 9125
@@
 Wire Wire Line
 	21850 12775 22175 12775
-Text Label 21300 12775 2    50   ~ 0
-GRND
 Wire Wire Line
 	23500 11975 23500 11250
@@
 Wire Wire Line
 	19900 17525 21250 17525
-Text Label 21250 17525 0    50   ~ 0
-~RD
 Wire Wire Line
 	19900 17425 21250 17425
@@
 Wire Wire Line
 	19900 17325 21250 17325
-Text Label 21250 17325 0    50   ~ 0
-~WR
 Wire Wire Line
 	19900 16525 19950 16525
@@
 	0    1    -1   0
 $EndComp
-Text Label 19050 16525 2    50   ~ 0
-TDI
-Text Label 19900 17075 0    50   ~ 0
-TDO
 $Comp
 L Device:R R112
@@
 Wire Wire Line
 	19775 11825 19875 11825
-Text Label 19625 11825 2    50   ~ 0
-GRND
 Wire Wire Line
 	19900 16625 21775 16625
@@
 	1    0    0    -1
 $EndComp
-Text Label 22925 15500 0    50   ~ 0
-~TM1
 $Comp
 L 74xx:74LS00 U418
@@
 	1    0    0    -1
 $EndComp
-Text Label 22925 14725 0    50   ~ 0
-~TM2
 Wire Wire Line
 	21775 15600 21700 15600
@@
 Wire Wire Line
 	5575 17625 5625 17625
-Text Label 5575 17750 3    50   ~ 0
-RD0
 Wire Wire Line
 	5500 17525 5500 17750
@@
 Wire Wire Line
 	5350 17325 4950 17325
-Text Label 5500 17750 3    50   ~ 0
-RD1
-Text Label 5425 17750 3    50   ~ 0
-RD2
-Text Label 5350 17750 3    50   ~ 0
-RD3
-Text Label 5275 17750 3    50   ~ 0
-RD4
-Text Label 5200 17750 3    50   ~ 0
-RD5
-Text Label 5125 17750 3    50   ~ 0
-RD6
-Text Label 5050 17750 3    50   ~ 0
-RD7
 Connection ~ 5125 17025
 Wire Wire Line
@@
 	13775 19550 13775 19250
 Text Label 14175 19950 1    50   ~ 0
-~RFRSH
+~RFSH
 Wire Wire Line
 	14075 19950 13975 19950
-Text Label 13975 19950 1    50   ~ 0
-~MREQ
 Text Label 13975 20950 3    50   ~ 0
 ~ROM0
@@
 L power:GND #PWR0194
 U 1 1 62E944E8
-P 13650 20450
-F 0 "#PWR0194" H 13650 20200 50  0001 C CNN
-F 1 "GND" H 13675 20225 50  0000 C CNN
-F 2 "" H 13650 20450 50  0001 C CNN
-F 3 "" H 13650 20450 50  0001 C CNN
-	1    13650 20450
+P 13675 20450
+F 0 "#PWR0194" H 13675 20200 50  0001 C CNN
+F 1 "GND" H 13700 20225 50  0000 C CNN
+F 2 "" H 13675 20450 50  0001 C CNN
+F 3 "" H 13675 20450 50  0001 C CNN
+	1    13675 20450
 	0    1    1    0
 $EndComp
@@
 ~EXP1
 Text Label 12375 19925 1    50   ~ 0
-AB0
+AB-0
 Text Label 12275 19925 1    50   ~ 0
-AB1
+AB-1
 Text Label 12075 19925 1    50   ~ 0
-~EXP2
+~EXP0
 Text Label 11875 19925 1    50   ~ 0
-AB0
+AB-0
 Text Label 11775 19925 1    50   ~ 0
-AB1
+AB-1
 Text Label 9650 20925 3    50   ~ 0
 CTR
@@
 CIA
 Text Label 10250 20925 3    50   ~ 0
-EXP1
+~EXP1
 Text Label 10350 20925 3    50   ~ 0
-EXP0
+~EXP0
 Text Label 9850 20925 3    50   ~ 0
 ~VST
 Text Label 9950 20925 3    50   ~ 0
 ~ANIN
-Text Label 10050 20925 3    50   ~ 0
-~TVTL
 Text Label 10150 20925 3    50   ~ 0
 ~TVL
 Text Label 11775 20925 3    50   ~ 0
-~CLCSA
+~CLUSA
 Text Label 11875 20925 3    50   ~ 0
 ~ENRG2
@@
 ~CLDMA
 Text Label 12475 20925 3    50   ~ 0
-~COG
+~COP
 Text Label 12575 20925 3    50   ~ 0
 ~ENRG1
@@
 	1    0    0    -1
 $EndComp
-Text Label 8050 20500 0    50   ~ 0
-~INT
 Text Label 6250 20300 2    50   ~ 0
 ~CLK
@@
 	-1   0    0    1
 $EndComp
-Text Label 4975 7250 0    50   ~ 0
-~MREQ
 Text Label 4975 7150 0    50   ~ 0
 RAMINH
@@
 	-1   0    0    1
 $EndComp
-Text Label 6625 17825 0    50   ~ 0
-~RD
 Text Label 6625 17925 0    50   ~ 0
 ~CPRQG
@@
 ~RTSD
 Text GLabel 9725 19250 3    50   Input ~ 0
-D0
+DB-0
 Text GLabel 9525 19250 3    50   Input ~ 0
-P0
+PO
 Text GLabel 9925 19250 3    50   Input ~ 0
 ~CLK
@@
 TVP
 Text GLabel 9650 19925 1    50   Input ~ 0
-~IORQ
+~IOREQ
 Text GLabel 9025 18250 1    50   Input ~ 0
-~RST
+~RESET
 Text GLabel 10150 19925 1    50   Input ~ 0
-AB4
+AB-4
 Text GLabel 10250 19925 1    50   Input ~ 0
-AB3
+AB-3
 Text GLabel 10350 19925 1    50   Input ~ 0
-AB2
+AB-2
 Text GLabel 9750 19925 1    50   Input ~ 0
 PRTOV
@@
 Text Label 18125 3300 2    50   ~ 0
 ~ROM0
+NoConn ~ 14675 20950
+NoConn ~ 14575 20950
+NoConn ~ 14475 20950
+NoConn ~ 14375 20950
+NoConn ~ 14275 20950
+Text GLabel 22350 5500 1    50   Input ~ 0
+~M1
+Text GLabel 6750 1575 0    50   Input ~ 0
+~MREQ
+Text GLabel 13975 19950 1    50   Input ~ 0
+~MREQ
+Text GLabel 21250 17525 2    50   Input ~ 0
+~RD
+Text GLabel 21250 17325 2    50   Input ~ 0
+~WR
+Text GLabel 6625 17825 2    50   Input ~ 0
+~RD
+$Comp
+L power:GND #PWR0205
+U 1 1 5F3C26FF
+P 6125 18225
+F 0 "#PWR0205" H 6125 17975 50  0001 C CNN
+F 1 "GND" H 6150 18000 50  0000 C CNN
+F 2 "" H 6125 18225 50  0001 C CNN
+F 3 "" H 6125 18225 50  0001 C CNN
+	1    6125 18225
+	1    0    0    -1
+$EndComp
+Text GLabel 5050 17750 3    50   Input ~ 0
+RD7
+Text GLabel 5125 17750 3    50   Input ~ 0
+RD6
+Text GLabel 5200 17750 3    50   Input ~ 0
+RD5
+Text GLabel 5275 17750 3    50   Input ~ 0
+RD4
+Text GLabel 5350 17750 3    50   Input ~ 0
+RD3
+Text GLabel 5425 17750 3    50   Input ~ 0
+RD2
+Text GLabel 5500 17750 3    50   Input ~ 0
+RD1
+Text GLabel 5575 17750 3    50   Input ~ 0
+RD0
+NoConn ~ 14075 18250
+NoConn ~ 13975 18250
+Text GLabel 8050 20500 2    50   Input ~ 0
+~INT
+NoConn ~ 14075 19250
+Text GLabel 22925 15500 2    50   Input ~ 0
+~TM1
+Text GLabel 22925 14725 2    50   Input ~ 0
+~TM2
+NoConn ~ 11975 18250
+Text GLabel 10050 20925 3    50   Input ~ 0
+~TVTL
+$Comp
+L power:GND #PWR0208
+U 1 1 5FBB8C3A
+P 21300 10650
+F 0 "#PWR0208" H 21300 10400 50  0001 C CNN
+F 1 "GND" H 21325 10450 50  0000 C CNN
+F 2 "" H 21300 10650 50  0001 C CNN
+F 3 "" H 21300 10650 50  0001 C CNN
+	1    21300 10650
+	0    1    1    0
+$EndComp
+$Comp
+L power:GND #PWR0249
+U 1 1 5FCD22CF
+P 19625 11825
+F 0 "#PWR0249" H 19625 11575 50  0001 C CNN
+F 1 "GND" H 19650 11625 50  0000 C CNN
+F 2 "" H 19625 11825 50  0001 C CNN
+F 3 "" H 19625 11825 50  0001 C CNN
+	1    19625 11825
+	0    1    1    0
+$EndComp
+$Comp
+L power:GND #PWR0250
+U 1 1 5FD5DA69
+P 21300 12775
+F 0 "#PWR0250" H 21300 12525 50  0001 C CNN
+F 1 "GND" H 21325 12575 50  0000 C CNN
+F 2 "" H 21300 12775 50  0001 C CNN
+F 3 "" H 21300 12775 50  0001 C CNN
+	1    21300 12775
+	0    1    1    0
+$EndComp
+$Comp
+L power:GND #PWR0251
+U 1 1 5FDF392B
+P 19425 5800
+F 0 "#PWR0251" H 19425 5550 50  0001 C CNN
+F 1 "GND" H 19450 5600 50  0000 C CNN
+F 2 "" H 19425 5800 50  0001 C CNN
+F 3 "" H 19425 5800 50  0001 C CNN
+	1    19425 5800
+	0    -1   -1   0
+$EndComp
+Text GLabel 19050 16525 0    50   Input ~ 0
+TDI
+Text GLabel 19900 17075 2    50   Input ~ 0
+TDO
 $EndSCHEMATC

Commit message: Some more link fixes now below 100 warnings.
Signed-off-by: John Bradley <flypie@rocketmail.com>
Parts:
- added J1, J2, J3, J4: Conn_01x10, Connector_JST:JST_EH_S10B-EH_1x10_P2.50mm_Horizontal, symbol Connector_Generic:Conn_01x10
- added U446: 74LS21, Package_DIP:DIP-14_W7.62mm, symbol 74xx:74LS08
- added U449: 74LS157, Package_DIP:DIP-16_W7.62mm, symbol 74xx:74LS157_UNITS
Connections:
- net AB0 is gone; now on net AB-0: U431.13
- net 1.3M: now also J1.3 (Pin_3)
- net 1.4M: now also J1.4 (Pin_4)
- net 1.5M: now also J1.5 (Pin_5)
- net 1.6M: now also J1.6 (Pin_6)
- net 1\8c: now also C64.1, R62.1, U432.9, J1.2 (Pin_2)
- net 3.4M: now also J3.4 (Pin_4)
- net 3.5M: now also J3.5 (Pin_5)
- net 3.6M: now also J3.6 (Pin_6)
- net 80L: now also J1.9 (Pin_9)
- net CPRQ: now also J4.4 (Pin_4)
- net GND: now also U402.13 (I3b), U449.15 (E)
- net RAMINH: no longer R23.2, U426.5
- net RD0: now also J4.6 (Pin_6)
- net RD1: now also J4.7 (Pin_7)
- net RD2: now also J4.8 (Pin_8)
- net RD3: now also J1.1 (Pin_1)
- net RD4: now also J4.10 (Pin_10)
- net RD5: now also J2.10 (Pin_10)
- net RD6: now also J4.9 (Pin_9)
- net RD7: now also J4.3 (Pin_3)
- net ROW: now also J1.7 (Pin_7)
- net TVAD: now also J3.2 (Pin_2)
- net VCC: now also U425.10 (~PRE)
- net ~BUSAK: now also J2.8 (Pin_8)
- net ~CPRQG: now also J4.5 (Pin_5)
- net ~ENRG: no longer U427.5 (Q1)
- net ~RD: now also J4.2 (Pin_2)
- net ~RFSH: now also J2.7 (Pin_7)
- net ~TVCLK: now also J3.1 (Pin_1)
- net at U405.4 (I2a): now also U424.10 (CET), U425.9 (Q)
- net at U439.3, U441.4, U441.5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: no longer U441.11, U444.6 (I1b), U460.1 (C)
- net CIA renamed ~ACIA
- net ~AB-14M renamed ~A14M
- net ~A14M: now also J1.8 (Pin_8)
- new net: U441.11, U444.6 (I1b), U460.1 (C)
- new net: U446.3, U449.1 (S)
- new net 1\2: J3.3 (Pin_3)
- new net 1\4: J2.2 (Pin_2)
- new net 3.10M: J3.10 (Pin_10)
- new net 3.7M: J3.7 (Pin_7)
- new net 3.8M: J3.8 (Pin_8)
- new net 3.9M: J3.9 (Pin_9)
- new net 32\40: U446.2
- new net FCTR: J1.10 (Pin_10)
- new net FP: J2.5 (Pin_5)
- new net FRM: J2.3 (Pin_3)
- new net GR: U446.1
- new net LLVD: J2.6 (Pin_6)
- new net OG: U427.5 (Q1)
- new net RMSL: R23.2, U426.5
- new net TVSD: J4.1 (Pin_1)
- new net ~CSYNC: J2.4 (Pin_4)
- new net ~GR: J2.9 (Pin_9)
- new net ~TVS: J2.1 (Pin_1)
- no-connect marks 15 -> 17
Other:
- note added: "Sheet 2"
- moved on the sheet: U441B

Commit message: More Label fixing. Down to 16 Warnings. Lots of devie Labels and balues wrong.
Signed-off-by: John Bradley <flypie@rocketmail.com>
Parts:
- added J21: Conn_02x25_Top_Bottom, symbol Connector_Generic:Conn_02x25_Top_Bottom
- added J31: Conn_02x10_Top_Bottom, symbol Connector_Generic:Conn_02x10_Top_Bottom
- C23: renamed from C20; value 33pf -> 0.1
- C33: renamed from C13; value CP -> 47uf
- C5: renamed from C15; value 33pf -> 680pf
- C9: renamed from C21; value 33pf -> 0.1
- R10: renamed from R29; value 22 -> 4K7
- R14: renamed from R42; value 22 -> 41k2
- R15: renamed from R43; value 22 -> 39K
- R16: renamed from R32; value 22 -> 4K7
- R25: renamed from R39; value 22 -> 1.2k
- R3: renamed from R44; value 22 -> 150k
- renumbered C11 to C19, C14 to C29, Q8 to Q22, Q2 to Q8
Connections:
- net +5 is gone; now on net VCC: C22.1, C23.2, Q22.1 (E), R14.1
- net 1\16 is gone; now on net ~1\16: U459.1
- net AD1 is gone; now on net AB-1: U412.1 (S)
- net GO is gone; now on net GR: U462.1, U462.4
- net ~32\40 is gone; now on net 32\40: U427.10 (Q3)
- net ~VST is gone; now on net ~UST: U430.10 (O5)
- net +12I: no longer C18.2, R2.1
- net +5I: now also PWRIN1.6 (Pin_6)
- net -12I: now also C18.2, R2.1
- net AB-0: now also J21.20 (Pin_20)
- net AB-1: now also J21.19 (Pin_19)
- net AB-10: now also J21.12 (Pin_12)
- net AB-11: now also J21.11 (Pin_11)
- net AB-12: now also J21.15 (Pin_15)
- net AB-13: now also J21.4 (Pin_4)
- net AB-14: now also J21.3 (Pin_3)
- net AB-15: now also J21.39 (Pin_39)
- net AB-2: now also J21.18 (Pin_18)
- net AB-3: now also J21.17 (Pin_17)
- net AB-4: now also J21.37 (Pin_37)
- net AB-5: now also J21.25 (Pin_25)
- net AB-6: now also J21.26 (Pin_26)
- net AB-7: now also J21.16 (Pin_16)
- net AB-8: now also J21.13 (Pin_13)
- net AB-9: now also J21.14 (Pin_14)
- net DB-0: now also J21.21 (Pin_21); no longer U413.7 (Q2)
- net DB-1: now also J21.22 (Pin_22)
- net DB-2: now also J21.24 (Pin_24)
- net DB-3: now also J21.8 (Pin_8)
- net DB-4: now also J21.7 (Pin_7)
- net DB-5: now also J21.6 (Pin_6)
- net DB-6: now also J21.9 (Pin_9)
- net DB-7: now also J21.10 (Pin_10)
- net EXRM0: now also J21.30 (Pin_30)
- net EXRM1: now also J21.29 (Pin_29)
- net EXRM2: now also J21.28 (Pin_28)
- net FCTR: now also J21.23 (Pin_23)
- net GND: now also J21.1 (Pin_1), J31.10 (Pin_10)
- net K1: now also J31.1 (Pin_1)
- net K2: now also J31.2 (Pin_2)
- net K3: now also J31.3 (Pin_3)
- net K4: now also J31.4 (Pin_4)
- net K6: now also J31.6 (Pin_6)
- net K7: now also J31.7 (Pin_7)
- net K8: now also J31.8 (Pin_8)
- net K9: now also J31.9 (Pin_9)
- net PRTOV: now also J21.47 (Pin_47)
- net VCC: now also J31.5 (Pin_5); no longer PWRIN1.6 (Pin_6)
- net ~BUSAK: now also J21.38 (Pin_38)
- net ~BUSRQ: now also J21.33 (Pin_33)
- net ~FRMR: now also U422.1 (~MR), U423.1 (~MR)
- net ~HALT: now also J21.44 (Pin_44)
- net ~INT: now also J21.41 (Pin_41)
- net ~IOREQ: now also J21.46 (Pin_46)
- net ~MREQ: now also J21.45 (Pin_45)
- net ~NMI: now also J21.43 (Pin_43)
- net ~ROM0: now also U408.22 (OD)
- net ~WAIT: now also J21.36 (Pin_36)
- net at U403.4 (I2a), U424.11 (Q3), U443.13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: no longer U443.6, U444.10 (I1c), U444.2 (I0a)
- net at U422.2 (CP), U423.2 (CP): now also U424.2 (CP), U438.8
- net F5 renamed FS
- net OG: no longer names the net of U427.5 (Q1)
- net ~CSYNC renamed CSYNC
- new net: U443.6, U444.10 (I1c), U444.2 (I0a)
- new net DO: U413.7 (Q2)
- new net ~RST: J21.34 (Pin_34)
- no-connect marks 17 -> 54
Other:
- note removed: "Sheet 2"
