File: NewBrain Original KiCad/Two.sch (KiCad schematic (older format))
At the start: 123 parts, among them J1 Conn_01x10, J2 Conn_01x10, J21 Conn_02x25_Top_Bottom, J3 Conn_01x10, J31 Conn_02x10_Top_Bottom, J4 Conn_01x10, Q17 ZTX650, Q20 ZTX107, Q22 2n5193, Q49 BC546, Q66 2N3906, Q8 2n5193, U401 LM358, U402 74LS153, U403 74LS153, U404 74LS153, U405 74LS153, U406 2764, U407 NEC-PD2364, U408 NEC-PD23128, U409 Z80CPU-DIP, U412 74LS257, U413 74LS174, U417 MC14584BDG, U418 74LS00, U419 COP420L, U421 74LS06, U422 74LS161, U423 74LS161, U424 74LS161, U425 74LS74, U426 74LS86, U427 74LS174, U428 74LS257, U429 74LS139, U430 74LS138, U431 74LS32, U432 74LS04, U433 74LS32, U435 74LS06, U438 74LS08, U439 74LS04, U441 74LS00, U442 74LS138, U443 74LS11, U444 74LS157_UNITS, U445 74LS112, U446 74LS21, U449 74LS157, U452 MC14584BDG_UNITS, U459 74LS32, U460 74LS112, U462 74LS32, U464 74LS11, U465 74LS11, U470 74LS00, X48 Crystal

Commit message: Resolve inconsistencies in circuit diagram buy following traces.
Resistor name used twice temp solution add a and b to name.

Signed-off-by: John Bradley <flypie@rocketmail.com>
Parts:
- removed R25, R26, R54: 4K7, Resistor_THT:R_Axial_DIN0204_L3.6mm_D1.6mm_P1.90mm_Vertical, symbol Device:R
- removed R34, R35, R37, R38, R47, R48, R49, R50: 4k7, Resistor_THT:R_Axial_DIN0204_L3.6mm_D1.6mm_P1.90mm_Vertical, symbol Device:R
- added R50: 33pf, Capacitor_THT:C_Disc_D3.0mm_W1.6mm_P2.50mm, symbol Device:C
- added RN54: 4K7, Resistor_THT:R_Array_SIP9, symbol Device:R_Network08
- added RN59: R_Network08, Resistor_THT:R_Array_SIP9, symbol Device:R_Network08
- added unit 3 of U401
- C12: renamed from C16; value 33pf -> 680pf
- C18, C23, C9: value 0.1 -> 0.1uf
- C19, C29: value 33pf -> 0.1uf
- C26: renamed from C12; value 33pf -> 0.1uf
- C51: renamed from C17; value 33pf -> 27pF
- C55: renamed from C19; value 33pf -> 100pf
- C6: renamed from C23; value CP -> 22 uF
- C7: renamed from C22; value CP -> 47uf
- J1, J2, J3, J4: footprint Connector_JST:JST_EH_S10B-EH_1x10_P2.50mm_Horizontal -> Connector_JST:JST_EH_B10B-EH-A_1x10_P2.50mm_Vertical
- J21: footprint (none) -> Connector_PinHeader_2.54mm:PinHeader_2x25_P2.54mm_Vertical
- J31: value Conn_02x10_Top_Bottom -> Conn_01x12_Top_Bottom; footprint (none) -> Connector_JST:JST_EH_B12B-EH-A_1x12_P2.50mm_Vertical; symbol Connector_Generic:Conn_02x10_Top_Bottom -> Connector_Generic:Conn_01x12
- R28a1: renamed from R27; value 22 -> 28
- renumbered R31 to R11, R33 to R13, R28 to R27, R23 to R28b1, R46 to R4, R41 to R43, R36 to R52
Connections:
- net ~ENRG1 is gone; now on net ~ENRG: U429.9 (O3)
- net ~TVTL is gone; now on net ~TVCTL: U430.12 (O3)
- net +12: now also Q8.2 (C); no longer Q8.1 (E)
- net +12I: now also Q8.1 (E); no longer Q8.2 (C)
- net +5I: now also Q22.1 (E); no longer Q22.2 (C)
- net AB-15G: now also RN54.6 (R5)
- net DB-5: now also J21.5 (Pin_5); no longer J21.6 (Pin_6)
- net GND: now also R50.1, U401.4 (V-); no longer U402.12 (I2b), U402.13 (I3b), U422.11 (Q3)
- net RMSL: now also J21.6 (Pin_6)
- net VCC: now also Q22.2 (C), RN54.1 (common), RN59.1 (common); no longer Q22.1 (E)
- net ~BUSRQ: now also RN59.9 (R8)
- net ~COPINT: no longer U412.3 (I1a)
- net ~INT: now also RN59.7 (R6)
- net ~IOREQ: now also RN59.3 (R2)
- net ~MREQ: now also RN59.2 (R1)
- net ~NMI: now also RN59.8 (R7)
- net ~RD: now also RN59.4 (R3)
- net ~WAIT: now also RN59.6 (R5)
- net ~WR: now also RN59.5 (R4)
- net at U402.10 (I0b), U402.11 (I1b), U428.4 (Za)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: now also RN54.4 (R3)
- net at U402.5 (I1a), U428.7 (Zb), U442.2 (A1): now also RN54.7 (R6)
- net at Q49.1 (C), R40.2, R52.1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: now also R50.2
- net K11: now reaches J31.11 (Pin_11)
- net K12: now reaches J31.12 (Pin_12)
- net V0A: now reaches C29.2, C33.1, R28a1.2
- net V0A: now also U401.8 (V+)
- net RCO renamed RC0
- new net: U402.12 (I2b), U402.13 (I3b), U422.11 (Q3)
- new net RDDK: U412.3 (I1a)
- no-connect marks 54 -> 49
Other:
- moved on the sheet: C5, C64, Q66, R62, R63, R65, U432D

Commit message: Resolve diplicate R28 from drawings, one is R30 a pullup resistor connected.
Trace 4 pins on memory board header.

Add aligned PCB igmes with alpha channel and beginings of annotated image.


Signed-off-by: John Bradley <flypie@rocketmail.com>
Parts:
- R27: value 22 -> 4k7
- R28: renamed from R28a1; value 28 -> 100
- R30: renamed from R28b1; value 1K -> 4K7
- R32: renamed from R30; value 32 -> 56
Connections:
- net 3.10M is gone; now on net -5v: J3.10 (Pin_10)
- net 3.7M is gone; now on net GND: J3.7 (Pin_7)
- net 3.8M is gone; now on net VCC: J3.8 (Pin_8)
- net 3.9M is gone; now on net GND: J3.9 (Pin_9)
- no-connect marks 49 -> 45
Changed lines of the file:
@@
 P 21400 9425
 F 0 "R27" V 21625 9425 50  0000 C CNN
-F 1 "22" V 21525 9425 50  0000 C CNN
+F 1 "4k7" V 21525 9425 50  0000 C CNN
 F 2 "Resistor_THT:R_Axial_DIN0204_L3.6mm_D1.6mm_P1.90mm_Vertical" V 21330 9425 50  0001 C CNN
 F 3 "~" H 21400 9425 50  0001 C CNN
@@
 $EndComp
 $Comp
-L Device:R R28a1
+L Device:R R28
 U 1 1 604D581E
 P 20925 9275
-F 0 "R28a1" H 20850 9350 50  0000 R CNN
-F 1 "28" H 20850 9250 50  0000 R CNN
+F 0 "R28" H 20850 9350 50  0000 R CNN
+F 1 "100" H 20850 9250 50  0000 R CNN
 F 2 "Resistor_THT:R_Axial_DIN0204_L3.6mm_D1.6mm_P1.90mm_Vertical" V 20855 9275 50  0001 C CNN
 F 3 "~" H 20925 9275 50  0001 C CNN
@@
 $EndComp
 $Comp
-L Device:R R30
+L Device:R R32
 U 1 1 60580D76
 P 21850 9575
-F 0 "R30" H 21925 9625 50  0000 L CNN
-F 1 "32" H 21925 9575 50  0000 L CNN
+F 0 "R32" H 21925 9625 50  0000 L CNN
+F 1 "56" H 21925 9575 50  0000 L CNN
 F 2 "Resistor_THT:R_Axial_DIN0204_L3.6mm_D1.6mm_P1.90mm_Vertical" V 21780 9575 50  0001 C CNN
 F 3 "~" H 21850 9575 50  0001 C CNN
@@
 	4975 6975 4900 6975
 $Comp
-L Device:R R28b1
+L Device:R R30
 U 1 1 6432B780
 P 4750 6975
-F 0 "R28b1" V 4875 7000 50  0000 C CNN
-F 1 "1K" V 4975 7000 50  0000 C CNN
+F 0 "R30" V 4875 7000 50  0000 C CNN
+F 1 "4K7" V 4975 7000 50  0000 C CNN
 F 2 "Resistor_THT:R_Axial_DIN0204_L3.6mm_D1.6mm_P1.90mm_Vertical" V 4680 6975 50  0001 C CNN
 F 3 "~" H 4750 6975 50  0001 C CNN
@@
 Text Label 2300 13250 0    50   ~ 0
 3.6M
-Text Label 2300 13350 0    50   ~ 0
-3.7M
 Text Label 2300 13450 0    50   ~ 0
 3.8M
@@
 Text GLabel 17300 19250 3    50   Input ~ 0
 AB-1
-NoConn ~ 2300 13650
-NoConn ~ 2300 13550
-NoConn ~ 2300 13450
-NoConn ~ 2300 13350
 NoConn ~ 12075 20925
 Text Label 25550 3025 1    50   ~ 0
@@
 P 21300 9650
 F 0 "#FLG0104" H 21300 9725 50  0001 C CNN
-F 1 "PWR_FLAG" H 21300 9875 50  0000 C CNN
+F 1 "PWR_FLAG" H 21200 9775 50  0000 C CNN
 F 2 "" H 21300 9650 50  0001 C CNN
 F 3 "~" H 21300 9650 50  0001 C CNN
@@
 Wire Wire Line
 	21300 9650 21375 9650
+$Comp
+L power:GND #PWR0158
+U 1 1 5F1E9599
+P 2600 13350
+F 0 "#PWR0158" H 2600 13100 50  0001 C CNN
+F 1 "GND" V 2625 13175 50  0000 R CNN
+F 2 "" H 2600 13350 50  0001 C CNN
+F 3 "" H 2600 13350 50  0001 C CNN
+	1    2600 13350
+	0    -1   -1   0
+$EndComp
+$Comp
+L power:VCC #PWR0159
+U 1 1 5F1EE3A3
+P 2600 13450
+F 0 "#PWR0159" H 2600 13300 50  0001 C CNN
+F 1 "VCC" V 2600 13575 50  0000 L CNN
+F 2 "" H 2600 13450 50  0001 C CNN
+F 3 "" H 2600 13450 50  0001 C CNN
+	1    2600 13450
+	0    1    -1   0
+$EndComp
+$Comp
+L power:GND #PWR0160
+U 1 1 5F45C40E
+P 2575 13550
+F 0 "#PWR0160" H 2575 13300 50  0001 C CNN
+F 1 "GND" V 2600 13375 50  0000 R CNN
+F 2 "" H 2575 13550 50  0001 C CNN
+F 3 "" H 2575 13550 50  0001 C CNN
+	1    2575 13550
+	0    -1   -1   0
+$EndComp
+Text Label 2575 13650 0    50   ~ 0
+-5v
+Wire Wire Line
+	2300 13650 2575 13650
+Wire Wire Line
+	2575 13550 2300 13550
+Wire Wire Line
+	2600 13450 2300 13450
+Wire Wire Line
+	2600 13350 2300 13350
+Text Label 2300 13350 0    50   ~ 0
+3.7M
 $EndSCHEMATC
