File: NewBrain MainBoard Original KiCad/NewBrain Original.kicad_pcb (KiCad board)
At the start: 2 copper layers, 193 parts, among them J1 Conn_01x10, J11 Conn_02x03_Top_Bottom, J12 Conn_02x03_Top_Bottom, J13 Conn_02x03_Top_Bottom, J14 Conn_02x03_Top_Bottom, J2 Conn_01x10, J21 Conn_02x25_Top_Bottom, J3 Conn_01x10, J31 Conn_01x12_Top_Bottom, J4 Conn_01x10, Q100 ZTX107, Q110 ZTC212, Q17 ZTX650, Q20 ZTX107, Q22 2n5193, Q49 BC546, Q66 2N3906, Q8 2n5193, U107 IN914, U109 IN914, U401 LM358, U402 74LS153, U403 74LS153, U404 74LS153, U405 74LS153, U406 2764, U407 NEC-PD2364, U408 NEC-PD23128, U409 Z80CPU-DIP, U410 MC1489N, U411 MC1488N, U412 74LS257, U413 74LS174, U414 LM358, U415 HE721A0530, U416 HE751A0510, U417 MC14584BDG, U418 74LS00, U419 COP420L, U420 74LS374, U421 74LS06, U422 74LS161, U423 74LS161, U424 74LS161, U425 74LS74, U426 74LS86, U427 74LS174, U428 74LS257, U429 74LS139, U430 74LS138, U431 74LS32, U432 74LS04, U433 74LS32, U434 74LS86, U435 74LS06, U436 74LS166, U437 74LS08, U438 74LS08, U439 74LS04, U440 74LS02, U441 74LS00, U442 74LS138, U443 74LS11, U444 74LS157_UNITS, U445 74LS112, U446 74LS21, U447 74LS393, U448 74LS10, U449 74LS157, U450 74LS04, U451 SN74LS279AN, U452 MC14584BDG_UNITS, U453 2716-Memory_EPROM, U454 74LS166, U455 74LS27, U456 74LS32, U457 74LS10, U458 74LS90, U459 74LS32, U460 74LS112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

Commit message: Complete Expansion Port.
Signed-off-by: John Bradley <flypie@rocketmail.com>
Connections:
- C64 pad 1: /TWO/1\8c -> /TWO/1\8C
- J1 pad 2: /TWO/1\8c -> /TWO/1\8C
- J21 pad 2: Net-(J21-Pad2) -> /TWO/1\8C
- J21 pad 27: Net-(J21-Pad27) -> /TWO/~RAMENB
- J21 pad 31: Net-(J21-Pad31) -> /TWO/~ROMOV
- J21 pad 32: Net-(J21-Pad32) -> ~BUSRQ
- J21 pad 33: ~BUSRQ -> ~M1
- J21 pad 34: /TWO/~RST -> ~RESET
- J21 pad 35: Net-(J21-Pad35) -> /TWO/~RFSH
- J21 pad 40: Net-(J21-Pad40) -> ~WR
- J21 pad 42: Net-(J21-Pad42) -> ~RD
- J21 pad 48: Net-(J21-Pad48) -> /TWO/RAMINH
- J21 pad 49: Net-(J21-Pad49) -> VCC
- J21 pad 50: Net-(J21-Pad50) -> BUSRQ
- R62 pad 1: /TWO/1\8c -> /TWO/1\8C
- U431 pad 6: /ONE/BUSRQ -> BUSRQ
- U432 pad 10: /TWO/1\8c -> /TWO/1\8C
- U432 pad 9: /TWO/1\8c -> /TWO/1\8C
- U435 pad 11: /ONE/BUSRQ -> BUSRQ

Commit message: UPdates add links and fix values add smoothing capacitors.
Signed-off-by: John Bradley <flypie@rocketmail.com>
Parts:
- added C34: 0.1uF 50V, Capacitor_THT:C_Axial_L3.8mm_D2.6mm_P7.50mm_Horizontal, F.Cu at (319.4, 46.4)
- added C35: 0.1uF 50V, Capacitor_THT:C_Axial_L3.8mm_D2.6mm_P7.50mm_Horizontal, F.Cu at (319.4, 50.5)
- added C36: 0.1uF 50V, Capacitor_THT:C_Axial_L3.8mm_D2.6mm_P7.50mm_Horizontal, F.Cu at (330.1, 46.4)
- added C37: 0.1uF 50V, Capacitor_THT:C_Axial_L3.8mm_D2.6mm_P7.50mm_Horizontal, F.Cu at (319.4, 54.7)
- added C38: 0.1uF 50V, Capacitor_THT:C_Axial_L3.8mm_D2.6mm_P7.50mm_Horizontal, F.Cu at (330.1, 50.5)
- added C39: 0.1uF 50V, Capacitor_THT:C_Axial_L3.8mm_D2.6mm_P7.50mm_Horizontal, F.Cu at (319.4, 58.8)
- added C41: 0.1uF 50V, Capacitor_THT:C_Axial_L3.8mm_D2.6mm_P7.50mm_Horizontal, F.Cu at (340.7, 46.4)
- added C42: 0.1uF 50V, Capacitor_THT:C_Axial_L3.8mm_D2.6mm_P7.50mm_Horizontal, F.Cu at (330.1, 54.7)
- added C67: 0.1uF 50V, Capacitor_THT:C_Axial_L3.8mm_D2.6mm_P7.50mm_Horizontal, F.Cu at (340.7, 50.5)
- added C68: 0.1uF 50V, Capacitor_THT:C_Axial_L3.8mm_D2.6mm_P7.50mm_Horizontal, F.Cu at (330.1, 58.8)
- added C69: 0.1uF 50V, Capacitor_THT:C_Axial_L3.8mm_D2.6mm_P7.50mm_Horizontal, F.Cu at (340.7, 54.7)
- added C70: 0.1uF 50V, Capacitor_THT:C_Axial_L3.8mm_D2.6mm_P7.50mm_Horizontal, F.Cu at (340.7, 58.8)
- added J100: Conn_01x03, Connector_PinSocket_2.54mm:PinSocket_1x03_P2.54mm_Vertical, F.Cu at (304.8, 139.1)
- added J101: Conn_01x02, Connector_PinSocket_2.54mm:PinSocket_1x02_P2.54mm_Vertical, F.Cu at (309.4, 139.1)
- added J102: Conn_01x03, Connector_PinSocket_2.54mm:PinSocket_1x03_P2.54mm_Vertical, F.Cu at (356.9, 46.6)
- added J103: Conn_01x03, Connector_PinSocket_2.54mm:PinSocket_1x03_P2.54mm_Vertical, F.Cu at (361.5, 46.6)
- C104, C119, C125, C127, C94, C95: footprint Capacitor_THT:C_Disc_D3.0mm_W1.6mm_P2.50mm -> Capacitor_THT:CP_Radial_D4.0mm_P1.50mm
- C120: value 0.1 -> 0.1uF 50V; footprint Capacitor_THT:C_Disc_D3.0mm_W1.6mm_P2.50mm -> Capacitor_THT:C_Axial_L3.8mm_D2.6mm_P7.50mm_Horizontal
- C50: renamed from R50; value 33pf -> 100pf
- R11: value 32 -> 560
- R13: value 22 -> 4K7
- R27, R6: value 4k7 -> 4K7
- R43, R45: value 4K7 -> 47
- R62: value 12k -> 120
- RN134, RN59: value R_Network08 -> 4K7
- RN61: renamed from RN66; value R_Network03 -> 22K
- U421: value 74LS06 -> 74LS245
- renumbered R24 to R48
Connections:
- U408 pad 26: AB-13 -> Net-(J100-Pad2)
- U422 pad 1: ~FRMR -> Net-(J101-Pad2)
- U423 pad 1: ~FRMR -> Net-(J101-Pad2)
- U424 pad 1: ~FRMR -> Net-(J101-Pad2)
- U445 pad 14: ~FRMR -> Net-(J101-Pad2)
- U445 pad 15: ~FRMR -> Net-(J101-Pad2)
- U453 pad 18: UCR -> Net-(J102-Pad2)
