File: NewBrain MainBoard Original KiCad/One.sch (KiCad schematic (older format))
At the start: 94 parts, among them J11 Conn_02x03_Top_Bottom, J12 Conn_02x03_Top_Bottom, J13 Conn_02x03_Top_Bottom, J14 Conn_02x03_Top_Bottom, Q100 ZTX107, Q110 ZTC212, U107 IN914, U109 IN914, U410 MC1489N, U411 MC1488N, U414 LM358, U415 HE721A0530, U416 HE751A0510, U417 MC14584BDG, U420 74LS374, U426 74LS86, U431 74LS32, U433 74LS32, U434 74LS86, U435 74LS06, U436 74LS166, U437 74LS08, U438 74LS08, U439 74LS04, U440 74LS02, U441 74LS00, U446 74LS21, U447 74LS393, U448 74LS10, U449 74LS157, U450 74LS04, U451 SN74LS279AN, U453 2716-Memory_EPROM, U454 74LS166, U455 74LS27, U456 74LS32, U457 74LS10, U458 74LS90, U459 74LS32, U460 74LS112, U461 74LS95, U462 74LS32, U463 74LS32, U464 74LS11, U465 74LS11, U466 74LS21, U467 74LS04, U468 74LS393, U469 74LS10, U470 74LS00, U471 74LS11

Commit message: Complete Expansion Port.
Signed-off-by: John Bradley <flypie@rocketmail.com>
Changed lines of the file:
@@
 Wire Wire Line
 	8600 14625 8650 14625
-Text Label 8650 15025 0    50   ~ 0
-BUSRQ
 Wire Wire Line
 	6950 15125 6700 15125
@@
 Text GLabel 17375 2850 2    50   Input ~ 0
 V0A
+Text GLabel 8650 15025 2    50   Input ~ 0
+BUSRQ
 $EndSCHEMATC

Commit message: UPdates add links and fix values add smoothing capacitors.
Signed-off-by: John Bradley <flypie@rocketmail.com>
Parts:
- added J102, J103: Conn_01x03, Connector_PinSocket_2.54mm:PinSocket_1x03_P2.54mm_Vertical, symbol Connector_Generic:Conn_01x03
- C104, C119: footprint Capacitor_THT:C_Disc_D3.0mm_W1.6mm_P2.50mm -> Capacitor_THT:CP_Radial_D4.0mm_P1.50mm
- C120: value 0.1 -> 0.1uF 50V; footprint Capacitor_THT:C_Disc_D3.0mm_W1.6mm_P2.50mm -> Capacitor_THT:C_Axial_L3.8mm_D2.6mm_P7.50mm_Horizontal
- RN61: renamed from RN66; value R_Network03 -> 22K
Connections:
- net GND: now also J102.1 (Pin_1), J103.1 (Pin_1)
- net UCR: now also J102.3 (Pin_3), J103.3 (Pin_3); no longer U453.18 (~CE~/PGM)
- net at U453.21 (VPP): now also J103.2 (Pin_2)
- new net: J102.2 (Pin_2), U453.18 (~CE~/PGM)
- no-connect marks 21 -> 20
Changed lines of the file:
@@
 Text Label 3300 7100 0    50   ~ 0
 TXTQ
-NoConn ~ 1375 6425
 Wire Wire Line
 	2475 7000 1100 7000
@@
 F 0 "C104" H 15675 2725 50  0000 R CNN
 F 1 "47uf" H 15675 2825 50  0000 R CNN
-F 2 "Capacitor_THT:C_Disc_D3.0mm_W1.6mm_P2.50mm" H 15838 2650 50  0001 C CNN
+F 2 "Capacitor_THT:CP_Radial_D4.0mm_P1.50mm" H 15838 2650 50  0001 C CNN
 F 3 "~" H 15800 2800 50  0001 C CNN
 	1    15800 2800
@@
 P 19050 9425
 F 0 "C120" V 18775 9425 50  0000 C CNN
-F 1 "0.1" V 18875 9425 50  0000 C CNN
-F 2 "Capacitor_THT:C_Disc_D3.0mm_W1.6mm_P2.50mm" H 19088 9275 50  0001 C CNN
+F 1 "0.1uF 50V" V 18875 9425 50  0000 C CNN
+F 2 "Capacitor_THT:C_Axial_L3.8mm_D2.6mm_P7.50mm_Horizontal" H 19088 9275 50  0001 C CNN
 F 3 "~" H 19050 9425 50  0001 C CNN
 	1    19050 9425
@@
 F 0 "C119" V 18750 9725 50  0000 C CNN
 F 1 "47uf" V 18850 9725 50  0000 C CNN
-F 2 "Capacitor_THT:C_Disc_D3.0mm_W1.6mm_P2.50mm" H 19088 9575 50  0001 C CNN
+F 2 "Capacitor_THT:CP_Radial_D4.0mm_P1.50mm" H 19088 9575 50  0001 C CNN
 F 3 "~" H 19050 9725 50  0001 C CNN
 	1    19050 9725
@@
 Wire Wire Line
 	3450 4075 3450 4600
-Text Label 1375 6325 2    50   ~ 0
+Text Label 850  6350 0    50   ~ 0
 UCR
 NoConn ~ 7025 6050
@@
 	2500 7925 2500 7525
 $Comp
-L Device:R_Network03 RN66
+L Device:R_Network03 RN61
 U 1 1 62260EA2
 P 5300 7625
-F 0 "RN66" V 4925 7625 50  0000 C CNN
-F 1 "R_Network03" V 5025 7625 50  0000 C CNN
+F 0 "RN61" V 4925 7625 50  0000 C CNN
+F 1 "22K" V 5025 7625 50  0000 C CNN
 F 2 "Resistor_THT:R_Array_SIP5" V 5575 7625 50  0001 C CNN
 F 3 "http://www.vishay.com/docs/31509/csc.pdf" H 5300 7625 50  0001 C CNN
@@
 Text GLabel 8650 15025 2    50   Input ~ 0
 BUSRQ
+$Comp
+L Connector_Generic:Conn_01x03 J102
+U 1 1 5F51C9E8
+P 650 6450
+F 0 "J102" H 550 6100 50  0000 C CNN
+F 1 "Conn_01x03" H 550 6200 50  0000 C CNN
+F 2 "Connector_PinSocket_2.54mm:PinSocket_1x03_P2.54mm_Vertical" H 650 6450 50  0001 C CNN
+F 3 "~" H 650 6450 50  0001 C CNN
+	1    650  6450
+	-1   0    0    1
+$EndComp
+Wire Wire Line
+	1375 6325 1150 6325
+Wire Wire Line
+	1150 6325 1150 6450
+Wire Wire Line
+	1150 6450 850  6450
+$Comp
+L power:GND #PWR0201
+U 1 1 5F601A1E
+P 850 6550
+F 0 "#PWR0201" H 850 6300 50  0001 C CNN
+F 1 "GND" V 850 6375 50  0000 R CNN
+F 2 "" H 850 6550 50  0001 C CNN
+F 3 "" H 850 6550 50  0001 C CNN
+	1    850  6550
+	0    -1   -1   0
+$EndComp
+Text Label 850  6750 0    50   ~ 0
+UCR
+$Comp
+L Connector_Generic:Conn_01x03 J103
+U 1 1 5F603BC1
+P 650 6850
+F 0 "J103" H 550 6500 50  0000 C CNN
+F 1 "Conn_01x03" H 550 6600 50  0000 C CNN
+F 2 "Connector_PinSocket_2.54mm:PinSocket_1x03_P2.54mm_Vertical" H 650 6850 50  0001 C CNN
+F 3 "~" H 650 6850 50  0001 C CNN
+	1    650  6850
+	-1   0    0    1
+$EndComp
+Wire Wire Line
+	1150 6850 850  6850
+$Comp
+L power:GND #PWR0202
+U 1 1 5F603BCC
+P 850 6950
+F 0 "#PWR0202" H 850 6700 50  0001 C CNN
+F 1 "GND" V 850 6775 50  0000 R CNN
+F 2 "" H 850 6950 50  0001 C CNN
+F 3 "" H 850 6950 50  0001 C CNN
+	1    850  6950
+	0    -1   -1   0
+$EndComp
+Wire Wire Line
+	1150 6850 1150 6650
+Wire Wire Line
+	1150 6650 1375 6650
+Wire Wire Line
+	1375 6650 1375 6425
 $EndSCHEMATC
