File: NewBrain MainBoard Original KiCad/Two.sch (KiCad schematic (older format))
At the start: 115 parts, among them J1 Conn_01x10, J2 Conn_01x10, J21 Conn_02x25_Top_Bottom, J3 Conn_01x10, J31 Conn_01x12_Top_Bottom, J4 Conn_01x10, Q17 ZTX650, Q20 ZTX107, Q22 2n5193, Q49 BC546, Q66 2N3906, Q8 2n5193, U401 LM358, U402 74LS153, U403 74LS153, U404 74LS153, U405 74LS153, U406 2764, U407 NEC-PD2364, U408 NEC-PD23128, U409 Z80CPU-DIP, U412 74LS257, U413 74LS174, U417 MC14584BDG, U418 74LS00, U419 COP420L, U421 74LS06, U422 74LS161, U423 74LS161, U424 74LS161, U425 74LS74, U426 74LS86, U427 74LS174, U428 74LS257, U429 74LS139, U430 74LS138, U431 74LS32, U432 74LS04, U433 74LS32, U435 74LS06, U438 74LS08, U439 74LS04, U441 74LS00, U442 74LS138, U443 74LS11, U444 74LS157_UNITS, U445 74LS112, U446 74LS21, U449 74LS157, U452 MC14584BDG_UNITS, U459 74LS32, U460 74LS112, U462 74LS32, U464 74LS11, U465 74LS11, U470 74LS00, X48 Crystal

Commit message: Complete Expansion Port.
Signed-off-by: John Bradley <flypie@rocketmail.com>
Parts:
- J21: symbol Connector_Generic:Conn_02x25_Top_Bottom -> Connector_Generic:Conn_02x25_Odd_Even
Connections:
- net 1\8c is gone; now on net 1\8C: C64.1, J1.2 (Pin_2), R62.1, U432.10, U432.9
- net ~RST is gone; now on net ~RESET: J21.34 (Pin_34)
- net RAMINH: now also J21.48 (Pin_48)
- net VCC: now also J21.49 (Pin_49)
- net ~BUSRQ: now also J21.32 (Pin_32); no longer J21.33 (Pin_33)
- net ~M1: now also J21.33 (Pin_33)
- net ~RAMENB: now also J21.27 (Pin_27)
- net ~RD: now also J21.42 (Pin_42)
- net ~RFSH: now also J21.35 (Pin_35)
- net ~ROMOV: now also J21.31 (Pin_31)
- net ~WR: now also J21.40 (Pin_40)
- net 1\8C: now reaches J21.2 (Pin_2)
- net BUSRQ: now reaches J21.50 (Pin_50)
- no-connect marks 45 -> 34
Other:
- moved on the sheet: C12, C125, C127, C18, C19, C23, C26, C29, C33, C44, C5, C51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

Commit message: UPdates add links and fix values add smoothing capacitors.
Signed-off-by: John Bradley <flypie@rocketmail.com>
Parts:
- added J100: Conn_01x03, Connector_PinSocket_2.54mm:PinSocket_1x03_P2.54mm_Vertical, symbol Connector_Generic:Conn_01x03
- added J101: Conn_01x02, Connector_PinSocket_2.54mm:PinSocket_1x02_P2.54mm_Vertical, symbol Connector_Generic:Conn_01x02
- C125, C127, C94, C95: footprint Capacitor_THT:C_Disc_D3.0mm_W1.6mm_P2.50mm -> Capacitor_THT:CP_Radial_D4.0mm_P1.50mm
- C50: renamed from R50; value 33pf -> 100pf
- R11: value 32 -> 560
- R13: value 22 -> 4K7
- R27, R6: value 4k7 -> 4K7
- R43, R45: value 4K7 -> 47
- R62: value 12k -> 120
- RN134, RN59: value R_Network08 -> 4K7
- U421: value 74LS06 -> 74LS245
- renumbered R24 to R48
Connections:
- net AB-13: now also J100.3 (Pin_3); no longer U408.26 (A13)
- net VCC: now also J100.1 (Pin_1)
- net ~FRMR: now also J101.1 (Pin_1); no longer U422.1 (~MR), U423.1 (~MR), U424.1 (~MR), U445.14 (~R), U445.15 (~R)
- new net: J101.2 (Pin_2), U422.1 (~MR), U423.1 (~MR), U424.1 (~MR), U445.14 (~R), U445.15 (~R)
- new net: J100.2 (Pin_2), U408.26 (A13)
- no-connect marks 34 -> 33
Other:
- moved on the sheet: R48
Changed lines of the file:
@@
 U 1 1 5EE8CBFF
 P 2925 7200
-F 0 "U402" H 2925 5900 50  0000 C CNN
-F 1 "74LS153" H 2925 6000 50  0000 C CNN
+F 0 "U402" H 2750 6150 50  0000 C CNN
+F 1 "74LS153" H 2900 6000 50  0000 C CNN
 F 2 "Package_DIP:DIP-16_W7.62mm" H 2925 7200 50  0001 C CNN
 F 3 "http://www.ti.com/lit/gpn/sn74LS153" H 2925 7200 50  0001 C CNN
@@
 U 1 1 5EE8FAF1
 P 4125 5625
-F 0 "U422" V 4050 4750 50  0000 R CNN
-F 1 "74LS161" V 4150 4750 50  0000 R CNN
+F 0 "U422" V 4525 5350 50  0000 R CNN
+F 1 "74LS161" V 4525 5125 50  0000 R CNN
 F 2 "Package_DIP:DIP-16_W7.62mm" H 4125 5625 50  0001 C CNN
 F 3 "http://www.ti.com/lit/gpn/sn74LS161" H 4125 5625 50  0001 C CNN
@@
 P 2900 1700
 F 0 "R6" V 3025 1725 50  0000 C CNN
-F 1 "4k7" V 3125 1725 50  0000 C CNN
+F 1 "4K7" V 3125 1725 50  0000 C CNN
 F 2 "Resistor_THT:R_Axial_DIN0204_L3.6mm_D1.6mm_P1.90mm_Vertical" V 2830 1700 50  0001 C CNN
 F 3 "~" H 2900 1700 50  0001 C CNN
@@
 U 1 1 5F2E3FDF
 P 11575 2250
-F 0 "U406" H 11575 3475 50  0000 C CNN
-F 1 "2764" H 11575 3375 50  0000 C CNN
+F 0 "U406" H 11600 3450 50  0000 C CNN
+F 1 "2764" H 11600 3350 50  0000 C CNN
 F 2 "Package_DIP:DIP-28_W15.24mm" H 11575 2250 50  0001 C CNN
 F 3 "https://downloads.reactivemicro.com/Electronics/ROM/2764%20EPROM.pdf" H 11575 2250 50  0001 C CNN
@@
 	1    0    0    -1
 $EndComp
-Wire Wire Line
-	14900 2750 14675 2750
-Text GLabel 14675 2750 0    50   Input ~ 0
+Text GLabel 14200 3300 1    50   Input ~ 0
 AB-13
 $Comp
@@
 $EndComp
 Wire Wire Line
-	3250 5625 3250 6275
-Wire Wire Line
-	3250 5625 2875 5625
+	2950 5625 2575 5625
 Wire Wire Line
 	7600 5925 7600 6275
@@
 P 24075 7175
 F 0 "R62" V 23825 7175 50  0000 C CNN
-F 1 "12k" V 23925 7175 50  0000 C CNN
+F 1 "120" V 23925 7175 50  0000 C CNN
 F 2 "Resistor_THT:R_Axial_DIN0204_L3.6mm_D1.6mm_P1.90mm_Vertical" V 24005 7175 50  0001 C CNN
 F 3 "~" H 24075 7175 50  0001 C CNN
@@
 P 18175 9275
 F 0 "R27" V 18400 9275 50  0000 C CNN
-F 1 "4k7" V 18300 9275 50  0000 C CNN
+F 1 "4K7" V 18300 9275 50  0000 C CNN
 F 2 "Resistor_THT:R_Axial_DIN0204_L3.6mm_D1.6mm_P1.90mm_Vertical" V 18105 9275 50  0001 C CNN
 F 3 "~" H 18175 9275 50  0001 C CNN
@@
 P 18625 11550
 F 0 "R11" H 18700 11600 50  0000 L CNN
-F 1 "32" H 18700 11550 50  0000 L CNN
+F 1 "560" H 18700 11550 50  0000 L CNN
 F 2 "Resistor_THT:R_Axial_DIN0204_L3.6mm_D1.6mm_P1.90mm_Vertical" V 18555 11550 50  0001 C CNN
 F 3 "~" H 18625 11550 50  0001 C CNN
@@
 P 18950 12350
 F 0 "R13" H 19050 12425 50  0000 L CNN
-F 1 "22" H 19050 12325 50  0000 L CNN
+F 1 "4K7" H 19050 12325 50  0000 L CNN
 F 2 "Resistor_THT:R_Axial_DIN0204_L3.6mm_D1.6mm_P1.90mm_Vertical" V 18880 12350 50  0001 C CNN
 F 3 "~" H 18950 12350 50  0001 C CNN
@@
 F 0 "C94" H 19750 15575 50  0000 L CNN
 F 1 "47uf" H 19750 15475 50  0000 L CNN
-F 2 "Capacitor_THT:C_Disc_D3.0mm_W1.6mm_P2.50mm" H 19638 15350 50  0001 C CNN
+F 2 "Capacitor_THT:CP_Radial_D4.0mm_P1.50mm" H 19638 15350 50  0001 C CNN
 F 3 "~" H 19600 15500 50  0001 C CNN
 	1    19600 15500
@@
 F 0 "C95" H 19750 14775 50  0000 L CNN
 F 1 "47uf" H 19750 14725 50  0000 L CNN
-F 2 "Capacitor_THT:C_Disc_D3.0mm_W1.6mm_P2.50mm" H 19638 14575 50  0001 C CNN
+F 2 "Capacitor_THT:CP_Radial_D4.0mm_P1.50mm" H 19638 14575 50  0001 C CNN
 F 3 "~" H 19600 14725 50  0001 C CNN
 	1    19600 14725
@@
 F 0 "C127" V 20600 16375 50  0000 C CNN
 F 1 "10uf" V 20500 16375 50  0000 C CNN
-F 2 "Capacitor_THT:C_Disc_D3.0mm_W1.6mm_P2.50mm" H 20338 16250 50  0001 C CNN
+F 2 "Capacitor_THT:CP_Radial_D4.0mm_P1.50mm" H 20338 16250 50  0001 C CNN
 F 3 "~" H 20300 16400 50  0001 C CNN
 	1    20300 16400
@@
 F 0 "C125" V 20100 17850 50  0000 C CNN
 F 1 "10uf" V 20000 17850 50  0000 C CNN
-F 2 "Capacitor_THT:C_Disc_D3.0mm_W1.6mm_P2.50mm" H 20338 17700 50  0001 C CNN
+F 2 "Capacitor_THT:CP_Radial_D4.0mm_P1.50mm" H 20338 17700 50  0001 C CNN
 F 3 "~" H 20300 17850 50  0001 C CNN
 	1    20300 17850
@@
 P 19425 19050
 F 0 "R45" V 19675 19050 50  0000 C CNN
-F 1 "4K7" V 19575 19050 50  0000 C CNN
+F 1 "47" V 19575 19050 50  0000 C CNN
 F 2 "Resistor_THT:R_Axial_DIN0204_L3.6mm_D1.6mm_P1.90mm_Vertical" V 19355 19050 50  0001 C CNN
 F 3 "~" H 19425 19050 50  0001 C CNN
@@
 P 2900 17275
 F 0 "U421" H 2875 16350 50  0000 C CNN
-F 1 "74LS06" H 2875 16250 50  0000 C CNN
+F 1 "74LS245" H 2875 16250 50  0000 C CNN
 F 2 "Package_DIP:DIP-20_W7.62mm" H 2900 17275 50  0001 C CNN
 F 3 "http://www.ti.com/lit/gpn/sn74LS06" H 2900 17275 50  0001 C CNN
@@
 P 19875 20550
 F 0 "R43" V 19975 20500 50  0000 C CNN
-F 1 "4K7" V 19975 20700 50  0000 C CNN
+F 1 "47" V 19975 20700 50  0000 C CNN
 F 2 "Resistor_THT:R_Axial_DIN0204_L3.6mm_D1.6mm_P1.90mm_Vertical" V 19805 20550 50  0001 C CNN
 F 3 "~" H 19875 20550 50  0001 C CNN
@@
 P 4350 18325
 F 0 "RN134" H 3825 18250 50  0000 R CNN
-F 1 "R_Network08" H 3825 18350 50  0000 R CNN
+F 1 "4K7" H 3825 18350 50  0000 R CNN
 F 2 "Resistor_THT:R_Array_SIP9" V 4825 18325 50  0001 C CNN
 F 3 "http://www.vishay.com/docs/31509/csc.pdf" H 4350 18325 50  0001 C CNN
@@
 ~ROMOV
 $Comp
-L Device:R R24
+L Device:R R48
 U 1 1 6312FBD9
-P 10400 17850
-F 0 "R24" V 10500 17800 50  0000 C CNN
-F 1 "4K7" V 10500 18000 50  0000 C CNN
-F 2 "Resistor_THT:R_Axial_DIN0204_L3.6mm_D1.6mm_P1.90mm_Vertical" V 10330 17850 50  0001 C CNN
-F 3 "~" H 10400 17850 50  0001 C CNN
-	1    10400 17850
+P 10400 17675
+F 0 "R48" V 10500 17625 50  0000 C CNN
+F 1 "4K7" V 10500 17825 50  0000 C CNN
+F 2 "Resistor_THT:R_Axial_DIN0204_L3.6mm_D1.6mm_P1.90mm_Vertical" V 10330 17675 50  0001 C CNN
+F 3 "~" H 10400 17675 50  0001 C CNN
+	1    10400 17675
 	0    -1   1    0
 $EndComp
@@
 L power:VCC #PWR0203
 U 1 1 6312FBE3
-P 10550 17850
-F 0 "#PWR0203" H 10550 17700 50  0001 C CNN
-F 1 "VCC" V 10525 18025 50  0000 L CNN
-F 2 "" H 10550 17850 50  0001 C CNN
-F 3 "" H 10550 17850 50  0001 C CNN
-	1    10550 17850
+P 10550 17675
+F 0 "#PWR0203" H 10550 17525 50  0001 C CNN
+F 1 "VCC" V 10525 17850 50  0000 L CNN
+F 2 "" H 10550 17675 50  0001 C CNN
+F 3 "" H 10550 17675 50  0001 C CNN
+	1    10550 17675
 	0    1    1    0
 $EndComp
 Connection ~ 10250 17850
 Wire Wire Line
-	10250 17850 10250 17825
-Wire Wire Line
 	8350 18100 8350 17475
 Connection ~ 8350 17475
@@
 P 2925 6100
 F 0 "#PWR0206" H 2925 5850 50  0001 C CNN
-F 1 "GND" V 2950 5950 50  0000 R CNN
+F 1 "GND" H 3250 5925 50  0000 C CNN
 F 2 "" H 2925 6100 50  0001 C CNN
 F 3 "" H 2925 6100 50  0001 C CNN
@@
 	5300 4900 5675 4900
 Wire Wire Line
-	3250 5625 3250 4950
-Wire Wire Line
 	3250 4950 3625 4950
-Connection ~ 3250 5625
 Connection ~ 3625 4950
 Wire Wire Line
 	3625 4950 3625 5125
-Text GLabel 2875 5625 0    50   Input ~ 0
+Text GLabel 2575 5625 0    50   Input ~ 0
 ~FRMR
 Text GLabel 3025 20350 0    50   Input ~ 0
@@
 P 21725 5350
 F 0 "RN59" H 22125 5400 50  0000 L CNN
-F 1 "R_Network08" H 22125 5350 50  0000 L CNN
+F 1 "4K7" H 22125 5350 50  0000 L CNN
 F 2 "Resistor_THT:R_Array_SIP9" V 22300 5350 50  0001 C CNN
 F 3 "http://www.vishay.com/docs/31509/csc.pdf" H 21725 5350 50  0001 C CNN
@@
 Wire Wire Line
 	19300 5725 21325 5725
-NoConn ~ 22125 5550
 $Comp
-L Device:C R50
+L Device:C C50
 U 1 1 601DADD4
 P 20175 19275
-F 0 "R50" H 20050 19225 50  0000 R CNN
-F 1 "33pf" H 20050 19275 50  0000 R CNN
+F 0 "C50" H 20100 19350 50  0000 R CNN
+F 1 "100pf" H 20125 19425 50  0000 R CNN
 F 2 "Capacitor_THT:C_Disc_D3.0mm_W1.6mm_P2.50mm" H 20213 19125 50  0001 C CNN
 F 3 "~" H 20175 19275 50  0001 C CNN
@@
 Wire Wire Line
 	8650 16875 14250 16875
+$Comp
+L Connector_Generic:Conn_01x03 J100
+U 1 1 5F0968A4
+P 14300 3500
+F 0 "J100" V 14150 3700 50  0000 L CNN
+F 1 "Conn_01x03" V 14250 3700 50  0000 L CNN
+F 2 "Connector_PinSocket_2.54mm:PinSocket_1x03_P2.54mm_Vertical" H 14300 3500 50  0001 C CNN
+F 3 "~" H 14300 3500 50  0001 C CNN
+	1    14300 3500
+	0    1    1    0
+$EndComp
+Wire Wire Line
+	14300 3300 14300 2750
+Wire Wire Line
+	14300 2750 14900 2750
+$Comp
+L power:VCC #PWR0156
+U 1 1 5F134492
+P 14400 3300
+F 0 "#PWR0156" H 14400 3150 50  0001 C CNN
+F 1 "VCC" H 14425 3500 50  0000 C CNN
+F 2 "" H 14400 3300 50  0001 C CNN
+F 3 "" H 14400 3300 50  0001 C CNN
+	1    14400 3300
+	1    0    0    -1
+$EndComp
+$Comp
+L Connector_Generic:Conn_01x02 J101
+U 1 1 5F139AC4
+P 2950 5825
+F 0 "J101" V 2700 5825 50  0000 R CNN
+F 1 "Conn_01x02" V 2650 6125 50  0000 R CNN
+F 2 "Connector_PinSocket_2.54mm:PinSocket_1x02_P2.54mm_Vertical" H 2950 5825 50  0001 C CNN
+F 3 "~" H 2950 5825 50  0001 C CNN
+	1    2950 5825
+	0    -1   1    0
+$EndComp
+Wire Wire Line
+	3250 4950 3250 5625
+Wire Wire Line
+	3250 5625 3050 5625
+Connection ~ 3250 5625
+Wire Wire Line
+	3250 5625 3250 6275
+Wire Wire Line
+	10250 17625 10250 17675
+Connection ~ 10250 17675
+Wire Wire Line
+	10250 17675 10250 17850
 $EndSCHEMATC
